Commit message: no friction

File: cssdbot_description/ur10.urd2f.xacro (robot description, xacro)
@@ -74,4 +74,11 @@
       </xacro:cylinder_inertial>
     </link>
+    <gazebo reference="${prefix}base_link">
+      <kp>10000000.0</kp>
+      <kd>1.0</kd>
+      <mu1>1.0</mu1>
+      <mu2>1.0</mu2>
+      <minDepth>0.001</minDepth>
+    </gazebo>
     <joint name="${prefix}shoulder_pan_joint" type="revolute">
       <parent link="${prefix}base_link" />
@@ -87,4 +94,7 @@
       <dynamics damping="0.0" friction="0.0"/>
     </joint>
+    <gazebo reference="${prefix}shoulder_pan_joint">
+      <implicitSpringDamper>1</implicitSpringDamper>
+    </gazebo>
     <link name="${prefix}shoulder_link">
       <visual>
@@ -105,4 +115,11 @@
       </xacro:cylinder_inertial>
     </link>
+    <gazebo reference="${prefix}shoulder_link">
+      <kp>10000000.0</kp>
+      <kd>1.0</kd>
+      <mu1>1.0</mu1>
+      <mu2>1.0</mu2>
+      <minDepth>0.001</minDepth>
+    </gazebo>
     <joint name="${prefix}shoulder_lift_joint" type="revolute">
       <parent link="${prefix}shoulder_link" />
@@ -118,4 +135,7 @@
       <dynamics damping="0.0" friction="0.0"/>
     </joint>
+    <gazebo reference="${prefix}shoulder_lift_joint">
+      <implicitSpringDamper>1</implicitSpringDamper>
+    </gazebo>
     <link name="${prefix}upper_arm_link">
       <visual>
@@ -136,4 +156,11 @@
       </xacro:cylinder_inertial>
     </link>
+    <gazebo reference="${prefix}upper_arm_link">
+      <kp>10000000.0</kp>
+      <kd>1.0</kd>
+      <mu1>1.0</mu1>
+      <mu2>1.0</mu2>
+      <minDepth>0.001</minDepth>
+    </gazebo>
     <joint name="${prefix}elbow_joint" type="revolute">
       <parent link="${prefix}upper_arm_link" />
@@ -149,4 +176,7 @@
       <dynamics damping="0.0" friction="0.0"/>
     </joint>
+    <gazebo reference="${prefix}elbow_joint">
+      <implicitSpringDamper>1</implicitSpringDamper>
+    </gazebo>
     <link name="${prefix}forearm_link">
       <visual>
@@ -167,4 +197,11 @@
       </xacro:cylinder_inertial>
     </link>
+    <gazebo reference="${prefix}forearm_link">
+      <kp>10000000.0</kp>
+      <kd>1.0</kd>
+      <mu1>1.0</mu1>
+      <mu2>1.0</mu2>
+      <minDepth>0.001</minDepth>
+    </gazebo>
     <joint name="${prefix}wrist_1_joint" type="revolute">
       <parent link="${prefix}forearm_link" />
@@ -180,4 +217,7 @@
       <dynamics damping="0.0" friction="0.0"/>
     </joint>
+    <gazebo reference="${prefix}wrist_1_joint">
+      <implicitSpringDamper>1</implicitSpringDamper>
+    </gazebo>
     <link name="${prefix}wrist_1_link">
       <visual>
@@ -198,4 +238,11 @@
       </xacro:cylinder_inertial>
     </link>
+    <gazebo reference="${prefix}wrist_1_link">
+      <kp>10000000.0</kp>
+      <kd>1.0</kd>
+      <mu1>1.0</mu1>
+      <mu2>1.0</mu2>
+      <minDepth>0.001</minDepth>
+    </gazebo>
     <joint name="${prefix}wrist_2_joint" type="revolute">
       <parent link="${prefix}wrist_1_link" />
@@ -211,4 +258,7 @@
       <dynamics damping="0.0" friction="0.0"/>
     </joint>
+    <gazebo reference="${prefix}wrist_2_joint">
+      <implicitSpringDamper>1</implicitSpringDamper>
+    </gazebo>
     <link name="${prefix}wrist_2_link">
       <visual>
@@ -229,4 +279,11 @@
       </xacro:cylinder_inertial>
     </link>
+    <gazebo reference="${prefix}wrist_2_link">
+      <kp>10000000.0</kp>
+      <kd>1.0</kd>
+      <mu1>1.0</mu1>
+      <mu2>1.0</mu2>
+      <minDepth>0.001</minDepth>
+    </gazebo>
     <joint name="${prefix}wrist_3_joint" type="revolute">
       <parent link="${prefix}wrist_2_link" />
@@ -242,4 +299,7 @@
       <dynamics damping="0.0" friction="0.0"/>
     </joint>
+    <gazebo reference="${prefix}wrist_3_joint">
+      <implicitSpringDamper>1</implicitSpringDamper>
+    </gazebo>
     <link name="${prefix}wrist_3_link">
       <visual>
@@ -260,4 +320,11 @@
       </xacro:cylinder_inertial>
     </link>
+    <gazebo reference="${prefix}wrist_3_link">
+      <kp>10000000.0</kp>
+      <kd>1.0</kd>
+      <mu1>1.0</mu1>
+      <mu2>1.0</mu2>
+      <minDepth>0.001</minDepth>
+    </gazebo>
     <joint name="${prefix}ee_fixed_joint" type="fixed">
       <parent link="${prefix}wrist_3_link" />
@@ -265,4 +332,7 @@
       <origin xyz="0.0 ${wrist_3_length} 0.0" rpy="0.0 0.0 ${pi/2.0}" />
     </joint>
+    <gazebo reference="${prefix}ee_fixed_joint">
+      <implicitSpringDamper>1</implicitSpringDamper>
+    </gazebo>
     <link name="${prefix}ee_link">
       <collision>
@@ -273,4 +343,7 @@
       </collision>
     </link>
+    <gazebo reference="${prefix}ee_link">
+      <implicitSpringDamper>1</implicitSpringDamper>
+    </gazebo>
 <!--end effector-->
   <joint name="${prefix}end_effector_joint" type="fixed">
@@ -279,19 +352,22 @@
       <origin xyz="0.0 0.0 0.0" rpy="0.0 0 0.0" />
     </joint>
+    <gazebo reference="${prefix}end_effector_joint">
+      <implicitSpringDamper>1</implicitSpringDamper>
+    </gazebo>
     <link name="${prefix}end_effector_link">
       <visual>
         <geometry>
-          <mesh filename="package://cssdbot_description/meshes/visual/end_effector.STL" scale = "0.001 0.001 0.001"/>
-        </geometry>
-        <origin xyz="0.0 0.0 0.0" rpy="3.14 0 0" />
-        <material name="LightGrey">
-          <color rgba="0.7 0.7 0.7 1.0"/>
-        </material>
-      </visual>
-      <collision>
-        <geometry>
-          <mesh filename="package://cssdbot_description/meshes/collision/end_effector.STL" scale = "0.001 0.001 0.001"/>
-        </geometry>
-	<origin xyz="0.0 0.0 0.0" rpy="3.14 0 0" />
+          <mesh filename="package://cssdbot_description/meshes/visual/end_effector.STL"/>
+        </geometry>
+        <origin xyz="0.005 0.0 0.0" rpy="3.14 0 0" />
+        <material name="LightGrey">
+          <color rgba="0.7 0.7 0.7 1.0"/>
+        </material>
+      </visual>
+      <collision>
+        <geometry>
+          <mesh filename="package://cssdbot_description/meshes/collision/end_effector.STL"/>
+        </geometry>
+	<origin xyz="0.005 0.0 0.0" rpy="3.14 0.0 0" />
       </collision>
       <inertial>
@@ -304,35 +380,11 @@
       </xacro:cylinder_inertial> -->
     </link>
- <gazebo reference="${prefix}end_effector_link">
-   <mu1>1</mu1>
-   <mu2>1</mu2>
-   <fdir1>1 0 0</fdir1>
-   <maxContacts>1</maxContacts>
-   <minDepth>0.001</minDepth>
-   <gravity>true</gravity>
-   <collision name="eef_collision">
-     <geometry>
-        <mesh filename="package://cssdbot_description/meshes/visual/end_effector.STL" scale = "0.001 0.001 0.001"/>
-     </geometry>
-     <surface>
-       <friction>
-         <torsional>
-           <coefficient>10</coefficient>
-           <use_patch_radius>false</use_patch_radius>
-           <!-- should be the same as collision sphere radius -->
-           <surface_radius>0.02175</surface_radius>
-           <patch_radius>0.01</patch_radius>
-         </torsional>
-       </friction>
-       <contact>
-         <poissons_ratio>0.5</poissons_ratio>
-         <elastic_modulus>1e8</elastic_modulus>
-       </contact>
-     </surface>
-   </collision>
- </gazebo>
-<!-- <kd>1000000000</kd>
-    <minDepth>0</minDepth>
--->
+    <gazebo reference="${prefix}end_effector_link">
+      <kp>10000000.0</kp>
+      <kd>1.0</kd>
+      <mu1>1.0</mu1>
+      <mu2>1.0</mu2>
+      <minDepth>0.001</minDepth>
+    </gazebo>
 <!--end of end effector-->
 <!-- start of camera -->

File: cssdbot_description/ur10.urdf.xacro (robot description, xacro)
@@ -282,16 +282,16 @@
       <visual>
         <geometry>
-          <mesh filename="package://cssdbot_description/meshes/visual/end_effector.STL" scale = "0.001 0.001 0.001"/>
-        </geometry>
-        <origin xyz="0.0 0.0 0.0" rpy="3.14 0 0" />
-        <material name="LightGrey">
-          <color rgba="0.7 0.7 0.7 1.0"/>
-        </material>
-      </visual>
-      <collision>
-        <geometry>
-          <mesh filename="package://cssdbot_description/meshes/collision/end_effector.STL" scale = "0.001 0.001 0.001"/>
-        </geometry>
-	<origin xyz="0.0 0.0 0.0" rpy="3.14 0 0" />
+          <mesh filename="package://cssdbot_description/meshes/visual/end_effector.STL"/>
+        </geometry>
+        <origin xyz="0.005 0.0 0.0" rpy="3.14 0 0" />
+        <material name="LightGrey">
+          <color rgba="0.7 0.7 0.7 1.0"/>
+        </material>
+      </visual>
+      <collision>
+        <geometry>
+          <mesh filename="package://cssdbot_description/meshes/collision/end_effector.STL"/>
+        </geometry>
+	<origin xyz="0.005 0.0 0.0" rpy="3.14 0.0 0" />
       </collision>
       <inertial>
@@ -304,35 +304,4 @@
       </xacro:cylinder_inertial> -->
     </link>
- <gazebo reference="${prefix}end_effector_link">
-   <mu1>1</mu1>
-   <mu2>1</mu2>
-   <fdir1>1 0 0</fdir1>
-   <maxContacts>1</maxContacts>
-   <minDepth>0.001</minDepth>
-   <gravity>true</gravity>
-   <collision name="eef_collision">
-     <geometry>
-        <mesh filename="package://cssdbot_description/meshes/visual/end_effector.STL" scale = "0.001 0.001 0.001"/>
-     </geometry>
-     <surface>
-       <friction>
-         <torsional>
-           <coefficient>10</coefficient>
-           <use_patch_radius>false</use_patch_radius>
-           <!-- should be the same as collision sphere radius -->
-           <surface_radius>0.02175</surface_radius>
-           <patch_radius>0.01</patch_radius>
-         </torsional>
-       </friction>
-       <contact>
-         <poissons_ratio>0.5</poissons_ratio>
-         <elastic_modulus>1e8</elastic_modulus>
-       </contact>
-     </surface>
-   </collision>
- </gazebo>
-<!-- <kd>1000000000</kd>
-    <minDepth>0</minDepth>
--->
 <!--end of end effector-->
 <!-- start of camera -->

File: cssdbot_description/ur103.urdf.xacro (robot description, xacro)
@@ -87,4 +87,7 @@
       <dynamics damping="0.0" friction="0.0"/>
     </joint>
+    <gazebo reference="${prefix}shoulder_pan_joint">
+      <implicitSpringDamper>1</implicitSpringDamper>
+    </gazebo>
     <link name="${prefix}shoulder_link">
       <visual>
@@ -118,4 +121,7 @@
       <dynamics damping="0.0" friction="0.0"/>
     </joint>
+    <gazebo reference="${prefix}shoulder_lift_joint">
+      <implicitSpringDamper>1</implicitSpringDamper>
+    </gazebo>
     <link name="${prefix}upper_arm_link">
       <visual>
@@ -149,4 +155,7 @@
       <dynamics damping="0.0" friction="0.0"/>
     </joint>
+    <gazebo reference="${prefix}elbow_joint">
+      <implicitSpringDamper>1</implicitSpringDamper>
+    </gazebo>
     <link name="${prefix}forearm_link">
       <visual>
@@ -173,11 +182,14 @@
       <axis xyz="0 1 0" />
       <xacro:unless value="${joint_limited}">
-        <limit lower="${-2.0 * pi}" upper="${2.0 * pi}" effort="54.0" velocity="3.2"/>
-      </xacro:unless>
-      <xacro:if value="${joint_limited}">
-        <limit lower="${wrist_1_lower_limit}" upper="${wrist_1_upper_limit}" effort="54.0" velocity="3.2"/>
-      </xacro:if>
-      <dynamics damping="0.0" friction="0.0"/>
-    </joint>
+        <limit lower="${-2.0 * pi}" upper="${2.0 * pi}" effort="100.0" velocity="3.2"/>
+      </xacro:unless>
+      <xacro:if value="${joint_limited}">
+        <limit lower="${wrist_1_lower_limit}" upper="${wrist_1_upper_limit}" effort="100.0" velocity="3.2"/>
+      </xacro:if>
+      <dynamics damping="0.0" friction="0.0"/>
+    </joint>
+    <gazebo reference="${prefix}wrist_1_joint">
+      <implicitSpringDamper>1</implicitSpringDamper>
+    </gazebo>
     <link name="${prefix}wrist_1_link">
       <visual>
@@ -204,11 +216,14 @@
       <axis xyz="0 0 1" />
       <xacro:unless value="${joint_limited}">
-        <limit lower="${-2.0 * pi}" upper="${2.0 * pi}" effort="54.0" velocity="3.2"/>
-      </xacro:unless>
-      <xacro:if value="${joint_limited}">
-        <limit lower="${wrist_2_lower_limit}" upper="${wrist_2_upper_limit}" effort="54.0" velocity="3.2"/>
-      </xacro:if>
-      <dynamics damping="0.0" friction="0.0"/>
-    </joint>
+        <limit lower="${-2.0 * pi}" upper="${2.0 * pi}" effort="100.0" velocity="3.2"/>
+      </xacro:unless>
+      <xacro:if value="${joint_limited}">
+        <limit lower="${wrist_2_lower_limit}" upper="${wrist_2_upper_limit}" effort="100.0" velocity="3.2"/>
+      </xacro:if>
+      <dynamics damping="0.0" friction="0.0"/>
+    </joint>
+    <gazebo reference="${prefix}wrist_2_joint">
+      <implicitSpringDamper>1</implicitSpringDamper>
+    </gazebo>
     <link name="${prefix}wrist_2_link">
       <visual>
@@ -229,4 +244,11 @@
       </xacro:cylinder_inertial>
     </link>
+    <gazebo reference="${prefix}writst_2_link">
+      <kp>10000000.0</kp>
+      <kd>5.0</kd>
+      <mu1>1.0</mu1>
+      <mu2>1.0</mu2>
+      <minDepth>0.001</minDepth>
+    </gazebo>
     <joint name="${prefix}wrist_3_joint" type="revolute">
       <parent link="${prefix}wrist_2_link" />
@@ -235,11 +257,14 @@
       <axis xyz="0 1 0" />
       <xacro:unless value="${joint_limited}">
-        <limit lower="${-2.0 * pi}" upper="${2.0 * pi}" effort="54.0" velocity="3.2"/>
-      </xacro:unless>
-      <xacro:if value="${joint_limited}">
-        <limit lower="${wrist_3_lower_limit}" upper="${wrist_3_upper_limit}" effort="54.0" velocity="3.2"/>
-      </xacro:if>
-      <dynamics damping="0.0" friction="0.0"/>
-    </joint>
+        <limit lower="${-2.0 * pi}" upper="${2.0 * pi}" effort="100.0" velocity="3.2"/>
+      </xacro:unless>
+      <xacro:if value="${joint_limited}">
+        <limit lower="${wrist_3_lower_limit}" upper="${wrist_3_upper_limit}" effort="100.0" velocity="3.2"/>
+      </xacro:if>
+      <dynamics damping="0.0" friction="0.0"/>
+    </joint>
+    <gazebo reference="${prefix}wrist_3_joint">
+      <implicitSpringDamper>1</implicitSpringDamper>
+    </gazebo>
     <link name="${prefix}wrist_3_link">
       <visual>
@@ -260,4 +285,11 @@
       </xacro:cylinder_inertial>
     </link>
+    <gazebo reference="${prefix}writst_3_link">
+      <kp>10000000.0</kp>
+      <kd>5.0</kd>
+      <mu1>1.0</mu1>
+      <mu2>1.0</mu2>
+      <minDepth>0.001</minDepth>
+    </gazebo>
     <joint name="${prefix}ee_fixed_joint" type="fixed">
       <parent link="${prefix}wrist_3_link" />
@@ -265,4 +297,7 @@
       <origin xyz="0.0 ${wrist_3_length} 0.0" rpy="0.0 0.0 ${pi/2.0}" />
     </joint>
+    <gazebo reference="${prefix}ee_fixed_joint">
+      <implicitSpringDamper>1</implicitSpringDamper>
+    </gazebo>
     <link name="${prefix}ee_link">
       <collision>
@@ -273,4 +308,14 @@
       </collision>
     </link>
+    <gazebo reference="${prefix}ee_link">
+      <kp>10000000.0</kp>
+      <kd>5.0</kd>
+      <mu1>1.0</mu1>
+      <mu2>1.0</mu2>
+      <minDepth>0.001</minDepth>
+    </gazebo>
+    <gazebo reference="${prefix}ee_link">
+      <implicitSpringDamper>1</implicitSpringDamper>
+    </gazebo>
 <!--end effector-->
   <joint name="${prefix}end_effector_joint" type="fixed">
@@ -279,19 +324,22 @@
       <origin xyz="0.0 0.0 0.0" rpy="0.0 0 0.0" />
     </joint>
+    <gazebo reference="${prefix}end_effector_joint">
+      <implicitSpringDamper>1</implicitSpringDamper>
+    </gazebo>
     <link name="${prefix}end_effector_link">
       <visual>
         <geometry>
-          <mesh filename="package://cssdbot_description/meshes/visual/end_effector.STL" scale = "0.001 0.001 0.001"/>
-        </geometry>
-        <origin xyz="0.0 0.0 0.0" rpy="3.14 0 0" />
-        <material name="LightGrey">
-          <color rgba="0.7 0.7 0.7 1.0"/>
-        </material>
-      </visual>
-      <collision>
-        <geometry>
-          <mesh filename="package://cssdbot_description/meshes/collision/end_effector.STL" scale = "0.001 0.001 0.001"/>
-        </geometry>
-	<origin xyz="0.0 0.0 0.0" rpy="3.14 0 0" />
+          <mesh filename="package://cssdbot_description/meshes/visual/end_effector.STL"/>
+        </geometry>
+        <origin xyz="0.005 0.0 0.0" rpy="3.14 0 0" />
+        <material name="LightGrey">
+          <color rgba="0.7 0.7 0.7 1.0"/>
+        </material>
+      </visual>
+      <collision>
+        <geometry>
+          <mesh filename="package://cssdbot_description/meshes/collision/end_effector.STL"/>
+        </geometry>
+	<origin xyz="0.005 0.0 0.0" rpy="3.14 0.0 0" />
       </collision>
       <inertial>
@@ -304,85 +352,13 @@
       </xacro:cylinder_inertial> -->
     </link>
- <gazebo reference="${prefix}end_effector_link">
-   <mu1>1</mu1>
-   <mu2>1</mu2>
-   <fdir1>1 0 0</fdir1>
-   <maxContacts>1</maxContacts>
-   <minDepth>0.001</minDepth>
-   <gravity>true</gravity>
-   <collision name="eef_collision">
-     <geometry>
-        <mesh filename="package://cssdbot_description/meshes/visual/end_effector.STL" scale = "0.001 0.001 0.001"/>
-     </geometry>
-     <surface>
-       <friction>
-         <torsional>
-           <coefficient>10</coefficient>
-           <use_patch_radius>false</use_patch_radius>
-           <!-- should be the same as collision sphere radius -->
-           <surface_radius>0.02175</surface_radius>
-           <patch_radius>0.01</patch_radius>
-         </torsional>
-       </friction>
-       <contact>
-         <poissons_ratio>0.5</poissons_ratio>
-         <elastic_modulus>1e8</elastic_modulus>
-       </contact>
-     </surface>
-   </collision>
- </gazebo>
-<!-- <kd>1000000000</kd>
-    <minDepth>0</minDepth>
--->
+    <gazebo reference="${prefix}end_effector_link">
+      <kp>10000000.0</kp>
+      <kd>5.0</kd>
+      <mu1>1.0</mu1>
+      <mu2>1.0</mu2>
+      <minDepth>0.001</minDepth>
+    </gazebo>
 <!--end of end effector-->
 <!-- start of camera -->
-  <joint name="camera_optical_joint" type="fixed">
-    <!-- satisfy both gazebo convention and aruco pkg convetion. looking from x axis and z axis respectively. -->
-    <origin xyz=" 0.055 0.06 0.0825" rpy="0 0.0 0" />>
-    <parent link="end_effector_link"/>
-    <child link="camera_link_optical"/>
-  </joint>
- <link name="camera_link_optical">
-  </link>
-<gazebo reference="camera_link_optical">
-    <sensor type="camera" name="camera1">
-      <update_rate>30.0</update_rate>
-      <camera name="camera_head">
-        <horizontal_fov>1.57</horizontal_fov>
-        <image>
-          <width>3840</width>
-          <height>1080</height>
-          <!--<format>R8G8B8</format> -->
-          <format>R8G8B8</format>
-        </image>
-        <clip>
-          <near>0.02</near>
-          <far>300</far>
-        </clip>
-        <noise>
-          <type>gaussian</type>
-          <!-- Noise is sampled independently per pixel on each frame.
-               That pixel's noise value is added to each of its color
-               channels, which at that point lie in the range [0,1]. -->
-          <mean>0.0</mean>
-          <stddev>0.007</stddev>
-        </noise>
-      </camera>
-      <plugin name="camera_controller" filename="libgazebo_ros_camera.so">
-        <alwaysOn>true</alwaysOn>
-        <updateRate>30</updateRate>
-        <cameraName></cameraName>
-        <imageTopicName>/image</imageTopicName>
-        <cameraInfoTopicName>/camera_info</cameraInfoTopicName>
-        <frameName>camera_link</frameName>
-        <hackBaseline>0.07</hackBaseline>
-        <distortionK1>0.0</distortionK1>
-        <distortionK2>0.0</distortionK2>
-        <distortionK3>0.0</distortionK3>
-        <distortionT1>0.0</distortionT1>
-        <distortionT2>0.0</distortionT2>
-      </plugin>
-    </sensor>
-  </gazebo>
 <!--camera link-->
 <!--end of camera link-->
