Commit message: reorganize sub packages and all launch files

File: cssdbot_description/urdf/ur10.urdf.xacro (robot description, xacro)
@@ -282,5 +282,5 @@
       <visual>
         <geometry>
-          <mesh filename="package://cssd_ur_description/meshes/visual/end_effector.STL"/>
+          <mesh filename="package://cssdbot_description/meshes/visual/end_effector.STL"/>
         </geometry>
         <origin xyz="0.0 0.0 0.0" rpy="${-pi/2} 0.0 ${pi/2}" />
@@ -291,5 +291,5 @@
       <collision>
         <geometry>
-          <mesh filename="package://cssd_ur_description/meshes/collision/end_effector.STL"/>
+          <mesh filename="package://cssdbot_description/meshes/collision/end_effector.STL"/>
         </geometry>
 	<origin xyz="0.0 0.0 0.0" rpy="${-pi/2} 0.0 ${pi/2}" />

File: cssdbot_description/urdf/ur10_robot.urdf.xacro (robot description, xacro)
@@ -6,5 +6,5 @@
   <xacro:include filename="$(find ur_description)/urdf/common.gazebo.xacro" />
   <!-- ur10 -->
-  <xacro:include filename="$(find cssd_ur_description)/urdf/ur10.urdf.xacro" />
+  <xacro:include filename="$(find cssdbot_description)/urdf/ur10.urdf.xacro" />
   <!-- arm -->
   <xacro:ur10_robot prefix="" joint_limited="false"

Commit message: documentation

File: cssdbot_description/urdf/ur10.urdf.xacro (robot description, xacro)
@@ -293,4 +293,10 @@
           <mesh filename="package://cssdbot_description/meshes/collision/end_effector.STL" scale = "0.001 0.001 0.001"/>
         </geometry>
+        <surface>
+	  <friction>
+	    <ode>
+	    </ode>
+	  </friction>
+        </surface>
 	<origin xyz="0.0 0.0 0.0" rpy="3.14 0 0" />
       </collision>
@@ -304,9 +310,11 @@
       </xacro:cylinder_inertial> -->
     </link>
+<!--
  <gazebo reference="${prefix}end_effector_link">
-   <mu1>1</mu1>
-   <mu2>1</mu2>
-   <fdir1>1 0 0</fdir1>
-   <maxContacts>1</maxContacts>
+   <mu1 value="100000" />
+   <mu2 value="100000"/>
+   <kd value="0" />
+   <fdir>1 0 0 </fdir>
+   <maxContacts>100000</maxContacts>
    <minDepth>0.001</minDepth>
    <gravity>true</gravity>
@@ -320,5 +328,4 @@
            <coefficient>10</coefficient>
            <use_patch_radius>false</use_patch_radius>
-           <!-- should be the same as collision sphere radius -->
            <surface_radius>0.02175</surface_radius>
            <patch_radius>0.01</patch_radius>
@@ -331,5 +338,7 @@
      </surface>
    </collision>
+   <dynamics friction="100.0" />
  </gazebo>
+-->
 <!-- <kd>1000000000</kd>
     <minDepth>0</minDepth>

Commit message: Cleaning up simulation configuration files

File: cssdbot_description/urdf/ur10.urdf.xacro (robot description, xacro)
@@ -289,15 +289,28 @@
         </material>
       </visual>
+      <visual>
+        <geometry>
+          <!-- extents: ([0.0125, 0.281], [-0.114, 0.114], [-0.046, -0.043]) -->
+          <box size="0.2685 0.228 0.003" />
+        </geometry>
+        <origin xyz="0.14675 0.0 0.0445" rpy="0 0 0" />
+        <material name="LightGrey">
+          <color rgba="0.7 0.7 0.7 1.0"/>
+        </material>
+      </visual>
+      <!--
       <collision>
         <geometry>
           <mesh filename="package://cssdbot_description/meshes/collision/end_effector.STL" scale = "0.001 0.001 0.001"/>
         </geometry>
-        <surface>
-	  <friction>
-	    <ode>
-	    </ode>
-	  </friction>
-        </surface>
-	<origin xyz="0.0 0.0 0.0" rpy="3.14 0 0" />
+	      <origin xyz="0.0 0.0 0.0" rpy="3.14 0 0" />
+      </collision>
+      -->
+      <collision>
+        <geometry>
+          <!-- extents: ([0.0125, 0.281], [-0.114, 0.114], [-0.046, -0.043]) -->
+          <box size="0.2685 0.228 0.003" />
+        </geometry>
+        <origin xyz="0.14675 0.0 -0.0445" rpy="0 0 0" />
       </collision>
       <inertial>
@@ -311,31 +324,11 @@
     </link>
  <gazebo reference="${prefix}end_effector_link">
-   <mu1 value="100000" />
-   <mu2 value="100000"/>
-   <kd value="0" />
-   <fdir>1 0 0 </fdir>
-   <maxContacts>100000</maxContacts>
-   <minDepth>0.001</minDepth>
-   <gravity>true</gravity>
-   <collision name="eef_collision">
-     <geometry>
-        <mesh filename="package://cssdbot_description/meshes/visual/end_effector.STL" scale = "0.001 0.001 0.001"/>
-     </geometry>
-     <surface>
-       <friction>
-         <torsional>
-           <coefficient>10</coefficient>
-           <use_patch_radius>false</use_patch_radius>
-           <surface_radius>0.02175</surface_radius>
-           <patch_radius>0.01</patch_radius>
-         </torsional>
-       </friction>
-       <contact>
-         <poissons_ratio>0.5</poissons_ratio>
-         <elastic_modulus>1e8</elastic_modulus>
-       </contact>
-     </surface>
-   </collision>
-   <dynamics friction="100.0" />
+  <maxContacts>100000</maxContacts>
+  <gravity>true</gravity>
+  <collision name="eef_collision">
+    <geometry>
+      <mesh filename="package://cssdbot_description/meshes/visual/end_effector.STL" scale = "0.001 0.001 0.001"/>
+    </geometry>
+  </collision>
  </gazebo>
 <!-- <kd>1000000000</kd>

Commit message: Need to try using box primitives for end effector plate

File: cssdbot_description/urdf/ur10.urdf.xacro (robot description, xacro)
@@ -289,29 +289,33 @@
         </material>
       </visual>
-      <visual>
-        <geometry>
-          <!-- extents: ([0.0125, 0.281], [-0.114, 0.114], [-0.046, -0.043]) -->
+      <collision>
+        <geometry>
+          <mesh filename="package://cssdbot_description/meshes/collision/end_effector_holes.stl" scale = "1 1 1"/>
+        </geometry>
+	      <origin xyz="0.0 0.0 0.0" rpy="3.14 0 0" />
+      </collision>
+      <!-- extents: ([0.0125, 0.281], [-0.114, 0.114], [-0.046, -0.043]) -->
+      <!-- <visual>
+        <geometry>
+          <box size="0.2685 0.228 0.01" />
+        </geometry>
+        <origin xyz="0.14675 0.0 0.04" rpy="0 0 0" />
+        <material name="LightGrey">
+          <color rgba="0.7 0.7 0.7 1.0"/>
+        </material>
+      </visual>
+      <collision>
+        <geometry>
+          <box size="0.2685 0.228 0.01" />
+        </geometry>
+        <origin xyz="0.14675 0.0 0.04" rpy="0 0 0" />
+      </collision> -->
+      <!-- extents: ([0.0125, 0.281], [-0.114, 0.114], [-0.046, -0.043]) -->
+      <!-- <collision>
+        <geometry>
           <box size="0.2685 0.228 0.003" />
         </geometry>
         <origin xyz="0.14675 0.0 0.0445" rpy="0 0 0" />
-        <material name="LightGrey">
-          <color rgba="0.7 0.7 0.7 1.0"/>
-        </material>
-      </visual>
-      <!--
-      <collision>
-        <geometry>
-          <mesh filename="package://cssdbot_description/meshes/collision/end_effector.STL" scale = "0.001 0.001 0.001"/>
-        </geometry>
-	      <origin xyz="0.0 0.0 0.0" rpy="3.14 0 0" />
-      </collision>
-      -->
-      <collision>
-        <geometry>
-          <!-- extents: ([0.0125, 0.281], [-0.114, 0.114], [-0.046, -0.043]) -->
-          <box size="0.2685 0.228 0.003" />
-        </geometry>
-        <origin xyz="0.14675 0.0 -0.0445" rpy="0 0 0" />
-      </collision>
+      </collision> -->
       <inertial>
         <origin xyz="0.06804 0.002 -0.046" rpy="0 0 0"/>
@@ -323,5 +327,5 @@
       </xacro:cylinder_inertial> -->
     </link>
- <gazebo reference="${prefix}end_effector_link">
+ <!-- <gazebo reference="${prefix}end_effector_link">
   <maxContacts>100000</maxContacts>
   <gravity>true</gravity>
@@ -331,5 +335,5 @@
     </geometry>
   </collision>
- </gazebo>
+ </gazebo> -->
 <!-- <kd>1000000000</kd>
     <minDepth>0</minDepth>

File: cssdbot_description/urdf/ur10_robot.urdf.xacro (robot description, xacro)
@@ -15,5 +15,5 @@
     <parent link="world" />
     <child link = "base_link" />
-    <origin xyz="0.0 0.0 0.0" rpy="0.0 0.0 0.0" />
+    <origin xyz="0.0 0.0 0.005" rpy="0.0 0.0 0.0" />
   </joint>
 </robot>

Commit message: Cleanup models and launch files

File: cssdbot_description/urdf/ur10.urdf.xacro (robot description, xacro)
@@ -274,5 +274,5 @@
       </collision>
     </link>
-<!--end effector-->
+  <!--end effector-->
   <joint name="${prefix}end_effector_joint" type="fixed">
       <parent link="${prefix}ee_link" />
@@ -296,29 +296,20 @@
 	      <origin xyz="0.0 0.0 0.0" rpy="3.14 0 0" />
       </collision>
-      <!-- Extents: ([0.0125, 0.2112], +/- 0.5673, [-0.046, -0.043]) -->
+      <!-- Extents: ([0.0125, 0.2112], +/- 0.05673, [-0.046, -0.043]) -->
+      <!-- Note: I'm making this 3mm thicker than the actual model -->
+      <collision>
+        <origin xyz="0.11185 0.0 0.046"/>
+        <geometry>
+          <box size="0.1987 0.11346 0.006"/>
+        </geometry>
+      </collision>
       <!-- Extents: ([0.12276, 0.2112], +/- 0.08644, [-0.046, -0.043]) -->
-      <!-- extents: ([0.0125, 0.281], [-0.114, 0.114], [-0.046, -0.043]) -->
-      <!-- <visual>
-        <geometry>
-          <box size="0.2685 0.228 0.01" />
-        </geometry>
-        <origin xyz="0.14675 0.0 0.04" rpy="0 0 0" />
-        <material name="LightGrey">
-          <color rgba="0.7 0.7 0.7 1.0"/>
-        </material>
-      </visual>
-      <collision>
-        <geometry>
-          <box size="0.2685 0.228 0.01" />
-        </geometry>
-        <origin xyz="0.14675 0.0 0.04" rpy="0 0 0" />
-      </collision> -->
-      <!-- extents: ([0.0125, 0.281], [-0.114, 0.114], [-0.046, -0.043]) -->
-      <!-- <collision>
-        <geometry>
-          <box size="0.2685 0.228 0.003" />
-        </geometry>
-        <origin xyz="0.14675 0.0 0.0445" rpy="0 0 0" />
-      </collision> -->
+      <!-- Note: I'm making this 3mm thicker than the actual model -->
+      <collision>
+        <origin xyz="0.16698 0.0 0.046"/>
+        <geometry>
+          <box size="0.08844 0.17288 0.006"/>
+        </geometry>
+      </collision>
       <inertial>
         <origin xyz="0.06804 0.002 -0.046" rpy="0 0 0"/>
