Commit message: ur10e option for arm 2

File: cssdbot_description/urdf/ur10/ur10_joint_limited_robot.urdf.xacro (robot description, xacro)
@@ -4,7 +4,7 @@
   <xacro:arg name="transmission_hw_interface" default="hardware_interface/PositionJointInterface"/>
   <!-- common stuff -->
-  <xacro:include filename="$(find ur_description)/urdf/common.gazebo.xacro" />
+  <xacro:include filename="$(find cssdbot_description)/urdf/ur10/common.gazebo.xacro" />
   <!-- ur10 -->
-  <xacro:include filename="$(find cssd_ur_description)/urdf/ur10.urdf.xacro" />
+  <xacro:include filename="$(find cssdbot_description)/urdf/ur10/ur10.urdf.xacro" />
   <!-- arm -->
   <xacro:ur10_robot prefix="" joint_limited="true"

File: cssdbot_description/urdf/ur10/ur10_robot.urdf.xacro (robot description, xacro)
@@ -4,7 +4,7 @@
   <xacro:arg name="transmission_hw_interface" default="hardware_interface/PositionJointInterface"/>
   <!-- common stuff -->
-  <xacro:include filename="$(find ur_description)/urdf/common.gazebo.xacro" />
+  <xacro:include filename="$(find cssdbot_description)/urdf/ur10/common.gazebo.xacro" />
   <!-- ur10 -->
-  <xacro:include filename="$(find cssdbot_description)/urdf/ur10.urdf.xacro" />
+  <xacro:include filename="$(find cssdbot_description)/urdf/ur10/ur10.urdf.xacro" />
   <!-- arm -->
   <xacro:ur10_robot prefix="" joint_limited="false"

File: cssdbot_description/urdf/ur10e/ur10e.urdf.xacro (robot description, xacro)
@@ -1,7 +1,6 @@
 <?xml version="1.0"?>
-<robot xmlns:xacro="http://wiki.ros.org/xacro">
-  <!-- <xacro:include filename="$(find cssdbot_description)/urdf/ur.transmission.xacro" /> -->
-  <xacro:include filename="$(find cssdbot_description)/urdf/ur.transmission.xacro" />
-  <xacro:include filename="$(find ur_description)/urdf/ur.gazebo.xacro" />
+<robot xmlns:xacro="http://ros.org/wiki/xacro">
+  <xacro:include filename="$(find cssdbot_description)/urdf/ur10e/ur.transmission.xacro" />
+  <xacro:include filename="$(find cssdbot_description)/urdf/ur10e/ur.gazebo.xacro" />
   <xacro:macro name="cylinder_inertial" params="radius length mass *origin">
     <inertial>
@@ -13,5 +12,5 @@
     </inertial>
   </xacro:macro>
-  <xacro:macro name="ur10_robot" params="prefix joint_limited
+  <xacro:macro name="ur10e_robot" params="prefix joint_limited
     shoulder_pan_lower_limit:=${-pi}    shoulder_pan_upper_limit:=${pi}
     shoulder_lift_lower_limit:=${-pi}    shoulder_lift_upper_limit:=${pi}
@@ -20,5 +19,7 @@
     wrist_2_lower_limit:=${-pi}    wrist_2_upper_limit:=${pi}
     wrist_3_lower_limit:=${-pi}    wrist_3_upper_limit:=${pi}
-    transmission_hw_interface:=hardware_interface/PositionJointInterface">
+    transmission_hw_interface:=hardware_interface/PositionJointInterface
+    safety_limits:=false safety_pos_margin:=0.15
+    safety_k_position:=20">
     <!-- Inertia parameters -->
     <xacro:property name="base_mass" value="4.0" />  <!-- This mass might be incorrect -->
@@ -31,5 +32,5 @@
     <!-- These parameters are borrowed from the urcontrol.conf file
         but are not verified for the correct permutation.
-        The permutation was guessed by looking at the UR5 parameters.
+        The permutation was guessed by looking at the ur5e parameters.
         Serious use of these parameters needs further inspection. -->
     <xacro:property name="shoulder_cog" value="0.00008 0.00244 -0.037" />
@@ -41,18 +42,18 @@
     <!-- Kinematic model -->
     <!-- Properties from urcontrol.conf -->
-    <xacro:property name="d1" value="0.1273" />
-    <xacro:property name="a2" value="-0.612" />
-    <xacro:property name="a3" value="-0.5723" />
-    <xacro:property name="d4" value="0.163941" />
-    <xacro:property name="d5" value="0.1157" />
-    <xacro:property name="d6" value="0.0922" />
+    <xacro:property name="d1" value="0.181" />
+    <xacro:property name="a2" value="-0.613" />
+    <xacro:property name="a3" value="-0.571" />
+    <xacro:property name="d4" value="0.135" />
+    <xacro:property name="d5" value="0.120" />
+    <xacro:property name="d6" value="0.117" />
     <!-- Arbitrary offsets for shoulder/elbow joints -->
-    <xacro:property name="shoulder_offset" value="0.220941" />  <!-- measured from model -->
-    <xacro:property name="elbow_offset" value="-0.1719" /> <!-- measured from model -->
+    <xacro:property name="shoulder_offset" value="0.176" />
+    <xacro:property name="elbow_offset" value="-0.137" />
     <!-- link lengths used in model -->
     <xacro:property name="shoulder_height" value="${d1}" />
     <xacro:property name="upper_arm_length" value="${-a2}" />
     <xacro:property name="forearm_length" value="${-a3}" />
-    <xacro:property name="wrist_1_length" value="${d4 - elbow_offset - shoulder_offset}" />
+    <xacro:property name="wrist_1_length" value="${d4}" />
     <xacro:property name="wrist_2_length" value="${d5}" />
     <xacro:property name="wrist_3_length" value="${d6}" />
@@ -60,13 +61,13 @@
       <visual>
         <geometry>
-          <mesh filename="package://ur_description/meshes/ur10/visual/base.dae"/>
-        </geometry>
-        <material name="LightGrey">
-          <color rgba="0.7 0.7 0.7 1.0"/>
-        </material>
-      </visual>
-      <collision>
-        <geometry>
-          <mesh filename="package://ur_description/meshes/ur10/collision/base.stl"/>
+          <mesh filename="package://ur_e_description/meshes/ur10e/visual/base.dae"/>
+        </geometry>
+        <material name="LightGrey">
+          <color rgba="0.7 0.7 0.7 1.0"/>
+        </material>
+      </visual>
+      <collision>
+        <geometry>
+          <mesh filename="package://ur_e_description/meshes/ur10e/collision/base.stl"/>
         </geometry>
       </collision>
@@ -81,8 +82,14 @@
       <axis xyz="0 0 1" />
       <xacro:unless value="${joint_limited}">
-        <limit lower="${-2.0 * pi}" upper="${2.0 * pi}" effort="330.0" velocity="2.16"/>
-      </xacro:unless>
-      <xacro:if value="${joint_limited}">
-        <limit lower="${shoulder_pan_lower_limit}" upper="${shoulder_pan_upper_limit}" effort="330.0" velocity="2.16"/>
+        <limit lower="${-2.0 * pi}" upper="${2.0 * pi}" effort="330.0" velocity="3.14"/>
+        <xacro:if value="${safety_limits}">
+          <safety_controller soft_lower_limit="${-2.0 * pi + safety_pos_margin}" soft_upper_limit="${2.0 * pi - safety_pos_margin}" k_position="${safety_k_position}" k_velocity="0.0"/>
+        </xacro:if>
+      </xacro:unless>
+      <xacro:if value="${joint_limited}">
+        <limit lower="${shoulder_pan_lower_limit}" upper="${shoulder_pan_upper_limit}" effort="330.0" velocity="3.14"/>
+        <xacro:if value="${safety_limits}">
+          <safety_controller soft_lower_limit="${shoulder_pan_lower_limit + safety_pos_margin}" soft_upper_limit="${shoulder_pan_upper_limit - safety_pos_margin}" k_position="${safety_k_position}" k_velocity="0.0"/>
+        </xacro:if>
       </xacro:if>
       <dynamics damping="0.0" friction="0.0"/>
@@ -91,13 +98,13 @@
       <visual>
         <geometry>
-          <mesh filename="package://ur_description/meshes/ur10/visual/shoulder.dae"/>
-        </geometry>
-        <material name="LightGrey">
-          <color rgba="0.7 0.7 0.7 1.0"/>
-        </material>
-      </visual>
-      <collision>
-        <geometry>
-          <mesh filename="package://ur_description/meshes/ur10/collision/shoulder.stl"/>
+          <mesh filename="package://ur_e_description/meshes/ur10e/visual/shoulder.dae"/>
+        </geometry>
+        <material name="LightGrey">
+          <color rgba="0.7 0.7 0.7 1.0"/>
+        </material>
+      </visual>
+      <collision>
+        <geometry>
+          <mesh filename="package://ur_e_description/meshes/ur10e/collision/shoulder.stl"/>
         </geometry>
       </collision>
@@ -112,8 +119,14 @@
       <axis xyz="0 1 0" />
       <xacro:unless value="${joint_limited}">
-        <limit lower="${-2.0 * pi}" upper="${2.0 * pi}" effort="330.0" velocity="2.16"/>
-      </xacro:unless>
-      <xacro:if value="${joint_limited}">
-        <limit lower="${shoulder_lift_lower_limit}" upper="${shoulder_lift_upper_limit}" effort="330.0" velocity="2.16"/>
+        <limit lower="${-2.0 * pi}" upper="${2.0 * pi}" effort="330.0" velocity="3.14"/>
+        <xacro:if value="${safety_limits}">
+          <safety_controller soft_lower_limit="${-2.0 * pi + safety_pos_margin}" soft_upper_limit="${2.0 * pi - safety_pos_margin}" k_position="${safety_k_position}" k_velocity="0.0"/>
+        </xacro:if>
+      </xacro:unless>
+      <xacro:if value="${joint_limited}">
+        <limit lower="${shoulder_lift_lower_limit}" upper="${shoulder_lift_upper_limit}" effort="330.0" velocity="3.14"/>
+        <xacro:if value="${safety_limits}">
+          <safety_controller soft_lower_limit="${shoulder_lift_lower_limit + safety_pos_margin}" soft_upper_limit="${shoulder_lift_upper_limit - safety_pos_margin}" k_position="${safety_k_position}" k_velocity="0.0"/>
+        </xacro:if>
       </xacro:if>
       <dynamics damping="0.0" friction="0.0"/>
@@ -122,13 +135,13 @@
       <visual>
         <geometry>
-          <mesh filename="package://ur_description/meshes/ur10/visual/upperarm.dae"/>
-        </geometry>
-        <material name="LightGrey">
-          <color rgba="0.7 0.7 0.7 1.0"/>
-        </material>
-      </visual>
-      <collision>
-        <geometry>
-          <mesh filename="package://ur_description/meshes/ur10/collision/upperarm.stl"/>
+          <mesh filename="package://ur_e_description/meshes/ur10e/visual/upperarm.dae"/>
+        </geometry>
+        <material name="LightGrey">
+          <color rgba="0.7 0.7 0.7 1.0"/>
+        </material>
+      </visual>
+      <collision>
+        <geometry>
+          <mesh filename="package://ur_e_description/meshes/ur10e/collision/upperarm.stl"/>
         </geometry>
       </collision>
@@ -143,8 +156,14 @@
       <axis xyz="0 1 0" />
       <xacro:unless value="${joint_limited}">
-        <limit lower="${-pi}" upper="${pi}" effort="150.0" velocity="3.15"/>
-      </xacro:unless>
-      <xacro:if value="${joint_limited}">
-        <limit lower="${elbow_joint_lower_limit}" upper="${elbow_joint_upper_limit}" effort="150.0" velocity="3.15"/>
+        <limit lower="${-pi}" upper="${pi}" effort="150.0" velocity="3.14"/>
+        <xacro:if value="${safety_limits}">
+          <safety_controller soft_lower_limit="${-2.0 * pi + safety_pos_margin}" soft_upper_limit="${2.0 * pi - safety_pos_margin}" k_position="${safety_k_position}" k_velocity="0.0"/>
+        </xacro:if>
+      </xacro:unless>
+      <xacro:if value="${joint_limited}">
+        <limit lower="${elbow_joint_lower_limit}" upper="${elbow_joint_upper_limit}" effort="150.0" velocity="3.14"/>
+        <xacro:if value="${safety_limits}">
+          <safety_controller soft_lower_limit="${elbow_joint_lower_limit + safety_pos_margin}" soft_upper_limit="${elbow_joint_upper_limit - safety_pos_margin}" k_position="${safety_k_position}" k_velocity="0.0"/>
+        </xacro:if>
       </xacro:if>
       <dynamics damping="0.0" friction="0.0"/>
@@ -153,13 +172,13 @@
       <visual>
          <geometry>
-          <mesh filename="package://ur_description/meshes/ur10/visual/forearm.dae"/>
-        </geometry>
-        <material name="LightGrey">
-          <color rgba="0.7 0.7 0.7 1.0"/>
-        </material>
-      </visual>
-      <collision>
-        <geometry>
-          <mesh filename="package://ur_description/meshes/ur10/collision/forearm.stl"/>
+          <mesh filename="package://ur_e_description/meshes/ur10e/visual/forearm.dae"/>
+        </geometry>
+        <material name="LightGrey">
+          <color rgba="0.7 0.7 0.7 1.0"/>
+        </material>
+      </visual>
+      <collision>
+        <geometry>
+          <mesh filename="package://ur_e_description/meshes/ur10e/collision/forearm.stl"/>
         </geometry>
       </collision>
@@ -174,8 +193,14 @@
       <axis xyz="0 1 0" />
       <xacro:unless value="${joint_limited}">
-        <limit lower="${-2.0 * pi}" upper="${2.0 * pi}" effort="54.0" velocity="3.2"/>
-      </xacro:unless>
-      <xacro:if value="${joint_limited}">
-        <limit lower="${wrist_1_lower_limit}" upper="${wrist_1_upper_limit}" effort="54.0" velocity="3.2"/>
+        <limit lower="${-2.0 * pi}" upper="${2.0 * pi}" effort="54.0" velocity="6.28"/>
+        <xacro:if value="${safety_limits}">
+          <safety_controller soft_lower_limit="${-2.0 * pi + safety_pos_margin}" soft_upper_limit="${2.0 * pi - safety_pos_margin}" k_position="${safety_k_position}" k_velocity="0.0"/>
+        </xacro:if>
+      </xacro:unless>
+      <xacro:if value="${joint_limited}">
+        <limit lower="${wrist_1_lower_limit}" upper="${wrist_1_upper_limit}" effort="54.0" velocity="6.28"/>
+        <xacro:if value="${safety_limits}">
+          <safety_controller soft_lower_limit="${wrist_1_lower_limit + safety_pos_margin}" soft_upper_limit="${wrist_1_upper_limit - safety_pos_margin}" k_position="${safety_k_position}" k_velocity="0.0"/>
+        </xacro:if>
       </xacro:if>
       <dynamics damping="0.0" friction="0.0"/>
@@ -184,17 +209,17 @@
       <visual>
         <geometry>
-          <mesh filename="package://ur_description/meshes/ur10/visual/wrist1.dae"/>
-        </geometry>
-        <material name="LightGrey">
-          <color rgba="0.7 0.7 0.7 1.0"/>
-        </material>
-      </visual>
-      <collision>
-        <geometry>
-          <mesh filename="package://ur_description/meshes/ur10/collision/wrist1.stl"/>
+          <mesh filename="package://ur_e_description/meshes/ur10e/visual/wrist1.dae"/>
+        </geometry>
+        <material name="LightGrey">
+          <color rgba="0.7 0.7 0.7 1.0"/>
+        </material>
+      </visual>
+      <collision>
+        <geometry>
+          <mesh filename="package://ur_e_description/meshes/ur10e/collision/wrist1.stl"/>
         </geometry>
       </collision>
       <xacro:cylinder_inertial radius="0.075" length="0.12" mass="${wrist_1_mass}">
-        <origin xyz="0.0 0.0 0.0" rpy="0 0 0" />
+        <origin xyz="0.0 ${wrist_1_length} 0.0" rpy="0 0 0" />
       </xacro:cylinder_inertial>
     </link>
@@ -205,8 +230,14 @@
       <axis xyz="0 0 1" />
       <xacro:unless value="${joint_limited}">
-        <limit lower="${-2.0 * pi}" upper="${2.0 * pi}" effort="54.0" velocity="3.2"/>
-      </xacro:unless>
-      <xacro:if value="${joint_limited}">
-        <limit lower="${wrist_2_lower_limit}" upper="${wrist_2_upper_limit}" effort="54.0" velocity="3.2"/>
+        <limit lower="${-2.0 * pi}" upper="${2.0 * pi}" effort="54.0" velocity="6.28"/>
+        <xacro:if value="${safety_limits}">
+          <safety_controller soft_lower_limit="${-2.0 * pi + safety_pos_margin}" soft_upper_limit="${2.0 * pi - safety_pos_margin}" k_position="${safety_k_position}" k_velocity="0.0"/>
+        </xacro:if>
+      </xacro:unless>
+      <xacro:if value="${joint_limited}">
+        <limit lower="${wrist_2_lower_limit}" upper="${wrist_2_upper_limit}" effort="54.0" velocity="6.28"/>
+        <xacro:if value="${safety_limits}">
+          <safety_controller soft_lower_limit="${wrist_2_lower_limit + safety_pos_margin}" soft_upper_limit="${wrist_2_upper_limit - safety_pos_margin}" k_position="${safety_k_position}" k_velocity="0.0"/>
+        </xacro:if>
       </xacro:if>
       <dynamics damping="0.0" friction="0.0"/>
@@ -215,17 +246,17 @@
       <visual>
         <geometry>
-          <mesh filename="package://ur_description/meshes/ur10/visual/wrist2.dae"/>
-        </geometry>
-        <material name="LightGrey">
-          <color rgba="0.7 0.7 0.7 1.0"/>
-        </material>
-      </visual>
-      <collision>
-        <geometry>
-          <mesh filename="package://ur_description/meshes/ur10/collision/wrist2.stl"/>
+          <mesh filename="package://ur_e_description/meshes/ur10e/visual/wrist2.dae"/>
+        </geometry>
+        <material name="LightGrey">
+          <color rgba="0.7 0.7 0.7 1.0"/>
+        </material>
+      </visual>
+      <collision>
+        <geometry>
+          <mesh filename="package://ur_e_description/meshes/ur10e/collision/wrist2.stl"/>
         </geometry>
       </collision>
       <xacro:cylinder_inertial radius="0.075" length="0.12" mass="${wrist_2_mass}">
-        <origin xyz="0.0 0.0 0.0" rpy="0 0 0" />
+        <origin xyz="0.0 0.0 ${wrist_2_length}" rpy="0 0 0" />
       </xacro:cylinder_inertial>
     </link>
@@ -236,8 +267,14 @@
       <axis xyz="0 1 0" />
       <xacro:unless value="${joint_limited}">
-        <limit lower="${-2.0 * pi}" upper="${2.0 * pi}" effort="54.0" velocity="3.2"/>
-      </xacro:unless>
-      <xacro:if value="${joint_limited}">
-        <limit lower="${wrist_3_lower_limit}" upper="${wrist_3_upper_limit}" effort="54.0" velocity="3.2"/>
+        <limit lower="${-2.0 * pi}" upper="${2.0 * pi}" effort="54.0" velocity="6.28"/>
+        <xacro:if value="${safety_limits}">
+          <safety_controller soft_lower_limit="${-2.0 * pi + safety_pos_margin}" soft_upper_limit="${2.0 * pi - safety_pos_margin}" k_position="${safety_k_position}" k_velocity="0.0"/>
+        </xacro:if>
+      </xacro:unless>
+      <xacro:if value="${joint_limited}">
+        <limit lower="${wrist_3_lower_limit}" upper="${wrist_3_upper_limit}" effort="54.0" velocity="6.28"/>
+        <xacro:if value="${safety_limits}">
+          <safety_controller soft_lower_limit="${wrist_3_lower_limit + safety_pos_margin}" soft_upper_limit="${wrist_3_upper_limit - safety_pos_margin}" k_position="${safety_k_position}" k_velocity="0.0"/>
+        </xacro:if>
       </xacro:if>
       <dynamics damping="0.0" friction="0.0"/>
@@ -246,17 +283,17 @@
       <visual>
         <geometry>
-          <mesh filename="package://ur_description/meshes/ur10/visual/wrist3.dae"/>
-        </geometry>
-        <material name="LightGrey">
-          <color rgba="0.7 0.7 0.7 1.0"/>
-        </material>
-      </visual>
-      <collision>
-        <geometry>
-          <mesh filename="package://ur_description/meshes/ur10/collision/wrist3.stl"/>
-        </geometry>
-      </collision>
-      <xacro:cylinder_inertial radius="0.075" length="0.12" mass="${wrist_3_mass}">
-        <origin xyz="0.0 0.0 0.0" rpy="0 0 0" />
+          <mesh filename="package://ur_e_description/meshes/ur10e/visual/wrist3.dae"/>
+        </geometry>
+        <material name="LightGrey">
+          <color rgba="0.7 0.7 0.7 1.0"/>
+        </material>
+      </visual>
+      <collision>
+        <geometry>
+          <mesh filename="package://ur_e_description/meshes/ur10e/collision/wrist3.stl"/>
+        </geometry>
+      </collision>
+      <xacro:cylinder_inertial radius="0.045" length="0.05" mass="${wrist_3_mass}">
+        <origin xyz="0.0 ${wrist_3_length - 0.05/2} 0.0" rpy="${pi/2} 0 0" />
       </xacro:cylinder_inertial>
     </link>
