Commit message: add ur10/ur10e meshes

File: cssdbot_description/urdf/ur10/ur10.urdf.xacro (robot description, xacro)
@@ -59,13 +59,13 @@
       <visual>
         <geometry>
-          <mesh filename="package://ur_description/meshes/ur10/visual/base.dae"/>
-        </geometry>
-        <material name="LightGrey">
-          <color rgba="0.7 0.7 0.7 1.0"/>
-        </material>
-      </visual>
-      <collision>
-        <geometry>
-          <mesh filename="package://ur_description/meshes/ur10/collision/base.stl"/>
+          <mesh filename="package://cssdbot_description/meshes/ur10/visual/base.dae"/>
+        </geometry>
+        <material name="LightGrey">
+          <color rgba="0.7 0.7 0.7 1.0"/>
+        </material>
+      </visual>
+      <collision>
+        <geometry>
+          <mesh filename="package://cssdbot_description/meshes/ur10/collision/base.stl"/>
         </geometry>
       </collision>
@@ -90,13 +90,13 @@
       <visual>
         <geometry>
-          <mesh filename="package://ur_description/meshes/ur10/visual/shoulder.dae"/>
-        </geometry>
-        <material name="LightGrey">
-          <color rgba="0.7 0.7 0.7 1.0"/>
-        </material>
-      </visual>
-      <collision>
-        <geometry>
-          <mesh filename="package://ur_description/meshes/ur10/collision/shoulder.stl"/>
+          <mesh filename="package://cssdbot_description/meshes/ur10/visual/shoulder.dae"/>
+        </geometry>
+        <material name="LightGrey">
+          <color rgba="0.7 0.7 0.7 1.0"/>
+        </material>
+      </visual>
+      <collision>
+        <geometry>
+          <mesh filename="package://cssdbot_description/meshes/ur10/collision/shoulder.stl"/>
         </geometry>
       </collision>
@@ -121,13 +121,13 @@
       <visual>
         <geometry>
-          <mesh filename="package://ur_description/meshes/ur10/visual/upperarm.dae"/>
-        </geometry>
-        <material name="LightGrey">
-          <color rgba="0.7 0.7 0.7 1.0"/>
-        </material>
-      </visual>
-      <collision>
-        <geometry>
-          <mesh filename="package://ur_description/meshes/ur10/collision/upperarm.stl"/>
+          <mesh filename="package://cssdbot_description/meshes/ur10/visual/upperarm.dae"/>
+        </geometry>
+        <material name="LightGrey">
+          <color rgba="0.7 0.7 0.7 1.0"/>
+        </material>
+      </visual>
+      <collision>
+        <geometry>
+          <mesh filename="package://cssdbot_description/meshes/ur10/collision/upperarm.stl"/>
         </geometry>
       </collision>
@@ -152,13 +152,13 @@
       <visual>
          <geometry>
-          <mesh filename="package://ur_description/meshes/ur10/visual/forearm.dae"/>
-        </geometry>
-        <material name="LightGrey">
-          <color rgba="0.7 0.7 0.7 1.0"/>
-        </material>
-      </visual>
-      <collision>
-        <geometry>
-          <mesh filename="package://ur_description/meshes/ur10/collision/forearm.stl"/>
+          <mesh filename="package://cssdbot_description/meshes/ur10/visual/forearm.dae"/>
+        </geometry>
+        <material name="LightGrey">
+          <color rgba="0.7 0.7 0.7 1.0"/>
+        </material>
+      </visual>
+      <collision>
+        <geometry>
+          <mesh filename="package://cssdbot_description/meshes/ur10/collision/forearm.stl"/>
         </geometry>
       </collision>
@@ -183,13 +183,13 @@
       <visual>
         <geometry>
-          <mesh filename="package://ur_description/meshes/ur10/visual/wrist1.dae"/>
-        </geometry>
-        <material name="LightGrey">
-          <color rgba="0.7 0.7 0.7 1.0"/>
-        </material>
-      </visual>
-      <collision>
-        <geometry>
-          <mesh filename="package://ur_description/meshes/ur10/collision/wrist1.stl"/>
+          <mesh filename="package://cssdbot_description/meshes/ur10/visual/wrist1.dae"/>
+        </geometry>
+        <material name="LightGrey">
+          <color rgba="0.7 0.7 0.7 1.0"/>
+        </material>
+      </visual>
+      <collision>
+        <geometry>
+          <mesh filename="package://cssdbot_description/meshes/ur10/collision/wrist1.stl"/>
         </geometry>
       </collision>
@@ -214,13 +214,13 @@
       <visual>
         <geometry>
-          <mesh filename="package://ur_description/meshes/ur10/visual/wrist2.dae"/>
-        </geometry>
-        <material name="LightGrey">
-          <color rgba="0.7 0.7 0.7 1.0"/>
-        </material>
-      </visual>
-      <collision>
-        <geometry>
-          <mesh filename="package://ur_description/meshes/ur10/collision/wrist2.stl"/>
+          <mesh filename="package://cssdbot_description/meshes/ur10/visual/wrist2.dae"/>
+        </geometry>
+        <material name="LightGrey">
+          <color rgba="0.7 0.7 0.7 1.0"/>
+        </material>
+      </visual>
+      <collision>
+        <geometry>
+          <mesh filename="package://cssdbot_description/meshes/ur10/collision/wrist2.stl"/>
         </geometry>
       </collision>
@@ -245,13 +245,13 @@
       <visual>
         <geometry>
-          <mesh filename="package://ur_description/meshes/ur10/visual/wrist3.dae"/>
-        </geometry>
-        <material name="LightGrey">
-          <color rgba="0.7 0.7 0.7 1.0"/>
-        </material>
-      </visual>
-      <collision>
-        <geometry>
-          <mesh filename="package://ur_description/meshes/ur10/collision/wrist3.stl"/>
+          <mesh filename="package://cssdbot_description/meshes/ur10/visual/wrist3.dae"/>
+        </geometry>
+        <material name="LightGrey">
+          <color rgba="0.7 0.7 0.7 1.0"/>
+        </material>
+      </visual>
+      <collision>
+        <geometry>
+          <mesh filename="package://cssdbot_description/meshes/ur10/collision/wrist3.stl"/>
         </geometry>
       </collision>
@@ -282,5 +282,5 @@
       <visual>
         <geometry>
-          <mesh filename="package://cssdbot_description/meshes/visual/end_effector.STL" scale = "0.001 0.001 0.001"/>
+          <mesh filename="package://cssdbot_description/meshes/end_effector/visual/end_effector.STL" scale = "0.001 0.001 0.001"/>
         </geometry>
         <origin xyz="0.0 0.0 0.0" rpy="3.14 0 0" />
@@ -291,5 +291,5 @@
       <collision>
         <geometry>
-          <mesh filename="package://cssdbot_description/meshes/collision/end_effector_holes.stl" scale = "1 1 1"/>
+          <mesh filename="package://cssdbot_description/meshes/end_effector/collision/end_effector_holes.stl" scale = "1 1 1"/>
         </geometry>
 	      <origin xyz="0.0 0.0 0.0" rpy="3.14 0 0" />
@@ -325,5 +325,5 @@
   <collision name="eef_collision">
     <geometry>
-      <mesh filename="package://cssdbot_description/meshes/visual/end_effector.STL" scale = "0.001 0.001 0.001"/>
+      <mesh filename="package://cssdbot_description/meshes/end_effector/visual/end_effector.STL" scale = "0.001 0.001 0.001"/>
     </geometry>
   </collision>

File: cssdbot_description/urdf/ur10e/ur10e.urdf.xacro (robot description, xacro)
@@ -61,13 +61,13 @@
       <visual>
         <geometry>
-          <mesh filename="package://ur_e_description/meshes/ur10e/visual/base.dae"/>
-        </geometry>
-        <material name="LightGrey">
-          <color rgba="0.7 0.7 0.7 1.0"/>
-        </material>
-      </visual>
-      <collision>
-        <geometry>
-          <mesh filename="package://ur_e_description/meshes/ur10e/collision/base.stl"/>
+          <mesh filename="package://cssdbot_description/meshes/ur10e/visual/base.dae"/>
+        </geometry>
+        <material name="LightGrey">
+          <color rgba="0.7 0.7 0.7 1.0"/>
+        </material>
+      </visual>
+      <collision>
+        <geometry>
+          <mesh filename="package://cssdbot_description/meshes/ur10e/collision/base.stl"/>
         </geometry>
       </collision>
@@ -98,13 +98,13 @@
       <visual>
         <geometry>
-          <mesh filename="package://ur_e_description/meshes/ur10e/visual/shoulder.dae"/>
-        </geometry>
-        <material name="LightGrey">
-          <color rgba="0.7 0.7 0.7 1.0"/>
-        </material>
-      </visual>
-      <collision>
-        <geometry>
-          <mesh filename="package://ur_e_description/meshes/ur10e/collision/shoulder.stl"/>
+          <mesh filename="package://cssdbot_description/meshes/ur10e/visual/shoulder.dae"/>
+        </geometry>
+        <material name="LightGrey">
+          <color rgba="0.7 0.7 0.7 1.0"/>
+        </material>
+      </visual>
+      <collision>
+        <geometry>
+          <mesh filename="package://cssdbot_description/meshes/ur10e/collision/shoulder.stl"/>
         </geometry>
       </collision>
@@ -135,13 +135,13 @@
       <visual>
         <geometry>
-          <mesh filename="package://ur_e_description/meshes/ur10e/visual/upperarm.dae"/>
-        </geometry>
-        <material name="LightGrey">
-          <color rgba="0.7 0.7 0.7 1.0"/>
-        </material>
-      </visual>
-      <collision>
-        <geometry>
-          <mesh filename="package://ur_e_description/meshes/ur10e/collision/upperarm.stl"/>
+          <mesh filename="package://cssdbot_description/meshes/ur10e/visual/upperarm.dae"/>
+        </geometry>
+        <material name="LightGrey">
+          <color rgba="0.7 0.7 0.7 1.0"/>
+        </material>
+      </visual>
+      <collision>
+        <geometry>
+          <mesh filename="package://cssdbot_description/meshes/ur10e/collision/upperarm.stl"/>
         </geometry>
       </collision>
@@ -172,13 +172,13 @@
       <visual>
          <geometry>
-          <mesh filename="package://ur_e_description/meshes/ur10e/visual/forearm.dae"/>
-        </geometry>
-        <material name="LightGrey">
-          <color rgba="0.7 0.7 0.7 1.0"/>
-        </material>
-      </visual>
-      <collision>
-        <geometry>
-          <mesh filename="package://ur_e_description/meshes/ur10e/collision/forearm.stl"/>
+          <mesh filename="package://cssdbot_description/meshes/ur10e/visual/forearm.dae"/>
+        </geometry>
+        <material name="LightGrey">
+          <color rgba="0.7 0.7 0.7 1.0"/>
+        </material>
+      </visual>
+      <collision>
+        <geometry>
+          <mesh filename="package://cssdbot_description/meshes/ur10e/collision/forearm.stl"/>
         </geometry>
       </collision>
@@ -209,13 +209,13 @@
       <visual>
         <geometry>
-          <mesh filename="package://ur_e_description/meshes/ur10e/visual/wrist1.dae"/>
-        </geometry>
-        <material name="LightGrey">
-          <color rgba="0.7 0.7 0.7 1.0"/>
-        </material>
-      </visual>
-      <collision>
-        <geometry>
-          <mesh filename="package://ur_e_description/meshes/ur10e/collision/wrist1.stl"/>
+          <mesh filename="package://cssdbot_description/meshes/ur10e/visual/wrist1.dae"/>
+        </geometry>
+        <material name="LightGrey">
+          <color rgba="0.7 0.7 0.7 1.0"/>
+        </material>
+      </visual>
+      <collision>
+        <geometry>
+          <mesh filename="package://cssdbot_description/meshes/ur10e/collision/wrist1.stl"/>
         </geometry>
       </collision>
@@ -246,13 +246,13 @@
       <visual>
         <geometry>
-          <mesh filename="package://ur_e_description/meshes/ur10e/visual/wrist2.dae"/>
-        </geometry>
-        <material name="LightGrey">
-          <color rgba="0.7 0.7 0.7 1.0"/>
-        </material>
-      </visual>
-      <collision>
-        <geometry>
-          <mesh filename="package://ur_e_description/meshes/ur10e/collision/wrist2.stl"/>
+          <mesh filename="package://cssdbot_description/meshes/ur10e/visual/wrist2.dae"/>
+        </geometry>
+        <material name="LightGrey">
+          <color rgba="0.7 0.7 0.7 1.0"/>
+        </material>
+      </visual>
+      <collision>
+        <geometry>
+          <mesh filename="package://cssdbot_description/meshes/ur10e/collision/wrist2.stl"/>
         </geometry>
       </collision>
@@ -283,13 +283,13 @@
       <visual>
         <geometry>
-          <mesh filename="package://ur_e_description/meshes/ur10e/visual/wrist3.dae"/>
-        </geometry>
-        <material name="LightGrey">
-          <color rgba="0.7 0.7 0.7 1.0"/>
-        </material>
-      </visual>
-      <collision>
-        <geometry>
-          <mesh filename="package://ur_e_description/meshes/ur10e/collision/wrist3.stl"/>
+          <mesh filename="package://cssdbot_description/meshes/ur10e/visual/wrist3.dae"/>
+        </geometry>
+        <material name="LightGrey">
+          <color rgba="0.7 0.7 0.7 1.0"/>
+        </material>
+      </visual>
+      <collision>
+        <geometry>
+          <mesh filename="package://cssdbot_description/meshes/ur10e/collision/wrist3.stl"/>
         </geometry>
       </collision>
@@ -320,5 +320,5 @@
       <visual>
         <geometry>
-          <mesh filename="package://cssdbot_description/meshes/visual/end_effector.STL" scale = "0.001 0.001 0.001"/>
+          <mesh filename="package://cssdbot_description/meshes/end_effector/visual/end_effector.STL" scale = "0.001 0.001 0.001"/>
         </geometry>
         <origin xyz="0.0 0.0 0.0" rpy="3.14 0 0" />
@@ -329,5 +329,5 @@
       <collision>
         <geometry>
-          <mesh filename="package://cssdbot_description/meshes/collision/end_effector_holes.stl" scale = "1 1 1"/>
+          <mesh filename="package://cssdbot_description/meshes/end_effector/collision/end_effector_holes.stl" scale = "1 1 1"/>
         </geometry>
 	      <origin xyz="0.0 0.0 0.0" rpy="3.14 0 0" />
@@ -363,5 +363,5 @@
   <collision name="eef_collision">
     <geometry>
-      <mesh filename="package://cssdbot_description/meshes/visual/end_effector.STL" scale = "0.001 0.001 0.001"/>
+      <mesh filename="package://cssdbot_description/meshes/end_effector/visual/end_effector.STL" scale = "0.001 0.001 0.001"/>
     </geometry>
   </collision>

File: cssdbot_description/urdf/ur10e/ur10e_robot.urdf.xacro (robot description, xacro)
@@ -2,5 +2,4 @@
 <robot xmlns:xacro="http://ros.org/wiki/xacro"
        name="ur10e" >
-  <xacro:arg name="transmission_hw_interface" default="hardware_interface/PositionJointInterface"/>
   <!-- common stuff -->
   <xacro:include filename="$(find cssdbot_description)/urdf/ur10e/common.gazebo.xacro" />
@@ -8,5 +7,5 @@
   <xacro:include filename="$(find cssdbot_description)/urdf/ur10e/ur10e.urdf.xacro" />
   <!-- arm -->
-  <xacro:ur10e_robot prefix="" joint_limited="false" transmission_hw_interface="$(arg transmission_hw_interface)"/>
+  <xacro:ur10e_robot prefix="" joint_limited="false" />
   <link name="world" />
   <joint name="world_joint" type="fixed">

Commit message: minimal dirty way namespace fix

File: cssdbot_description/urdf/ur10/ur10.urdf.xacro (robot description, xacro)
@@ -337,10 +337,10 @@
     <!-- satisfy both gazebo convention and aruco pkg convetion. looking from x axis and z axis respectively. -->
     <origin xyz=" 0.055 0.06 0.0825" rpy="0 0.0 0" />>
-    <parent link="end_effector_link"/>
-    <child link="camera_link_optical"/>
+    <parent link="${prefix}end_effector_link"/>
+    <child link="${prefix}camera_link_optical"/>
   </joint>
- <link name="camera_link_optical">
+ <link name="${prefix}camera_link_optical">
   </link>
-<gazebo reference="camera_link_optical">
+<gazebo reference="${prefix}camera_link_optical">
     <sensor type="camera" name="camera1">
       <update_rate>30.0</update_rate>
@@ -366,5 +366,5 @@
         </noise>
       </camera>
-      <plugin name="camera_controller" filename="libgazebo_ros_camera.so">
+      <plugin name="${prefix}camera_controller" filename="libgazebo_ros_camera.so">
         <alwaysOn>true</alwaysOn>
         <updateRate>30</updateRate>

File: cssdbot_description/urdf/ur10/ur10_joint_limited_robot.urdf.xacro (robot description, xacro)
@@ -3,4 +3,5 @@
        name="ur10" >
   <xacro:arg name="transmission_hw_interface" default="hardware_interface/PositionJointInterface"/>
+  <xacro:arg name="robot_ns" default=""/>
   <!-- common stuff -->
   <xacro:include filename="$(find cssdbot_description)/urdf/ur10/common.gazebo.xacro" />

File: cssdbot_description/urdf/ur10e/ur10e.urdf.xacro (robot description, xacro)
@@ -372,16 +372,16 @@
 <!--end of end effector-->
 <!-- start of camera -->
-  <joint name="camera_optical_joint" type="fixed">
+  <joint name="${prefix}camera_optical_joint" type="fixed">
     <!-- satisfy both gazebo convention and aruco pkg convetion. looking from x axis and z axis respectively. -->
     <origin xyz=" 0.055 0.06 0.0825" rpy="0 0.0 0" />>
-    <parent link="end_effector_link"/>
-    <child link="camera_link_optical"/>
+    <parent link="${prefix}end_effector_link"/>
+    <child link="${prefix}camera_link_optical"/>
   </joint>
- <link name="camera_link_optical">
+ <link name="${prefix}camera_link_optical">
   </link>
-<gazebo reference="camera_link_optical">
+<gazebo reference="${prefix}camera_link_optical">
     <sensor type="camera" name="camera1">
       <update_rate>30.0</update_rate>
-      <camera name="camera_head">
+      <camera name="${prefix}camera_head">
         <horizontal_fov>1.57</horizontal_fov>
         <image>
@@ -404,5 +404,6 @@
         </noise>
       </camera>
-      <plugin name="camera_controller" filename="libgazebo_ros_camera.so">
+      <plugin name="${prefix}camera_controller" filename="libgazebo_ros_camera.so">
+        <robotNamespace>$(arg robot_ns)</robotNamespace>
         <alwaysOn>true</alwaysOn>
         <updateRate>30</updateRate>

File: cssdbot_description/urdf/ur10e/ur10e_joint_limited_robot.urdf.xacro (robot description, xacro)
@@ -3,4 +3,5 @@
        name="ur10e" >
   <xacro:arg name="transmission_hw_interface" default="hardware_interface/PositionJointInterface"/>
+  <xacro:arg name="robot_ns" default=""/>
   <!-- common stuff -->
   <xacro:include filename="$(find cssdbot_description)/urdf/ur10e/common.gazebo.xacro" />
@@ -20,5 +21,5 @@
   <joint name="world_joint" type="fixed">
     <parent link="world" />
-    <child link = "base_link" />
+    <child link = "${robot_ns}base_link" />
     <origin xyz="0.0 0.0 0.0" rpy="0.0 0.0 0.0" />
   </joint>

File: cssdbot_description/urdf/ur10e/ur10e_robot.urdf.xacro (robot description, xacro)
@@ -1,13 +1,13 @@
 <?xml version="1.0"?>
-<robot xmlns:xacro="http://ros.org/wiki/xacro"
+<robot xmlns:xacro="http://wiki.ros.org/xacro"
        name="ur10e" >
   <xacro:arg name="transmission_hw_interface" default="hardware_interface/PositionJointInterface"/>
   <!-- common stuff -->
   <xacro:include filename="$(find cssdbot_description)/urdf/ur10e/common.gazebo.xacro" />
-  <!-- ur10e -->
-  <xacro:include filename="$(find cssdbot_description)/urdf/ur10e/ur10e.urdf.xacro" />
+  <!-- ur10 -->
+  <xacro:include filename="$(find cssdbot_description)/urdf/ur10/ur10e.urdf.xacro" />
   <!-- arm -->
-  <xacro:ur10e_robot prefix="" joint_limited="false"
-  transmission_hw_interface="$(arg transmission_hw_interface)"
+  <xacro:ur10_robot prefix="" joint_limited="false"
+    transmission_hw_interface="$(arg transmission_hw_interface)"
   />
   <link name="world" />

Commit message: fix image namespace

File: cssdbot_description/urdf/ur10/ur10.urdf.xacro (robot description, xacro)
@@ -370,6 +370,6 @@
         <updateRate>30</updateRate>
         <cameraName></cameraName>
-        <imageTopicName>/image</imageTopicName>
-        <cameraInfoTopicName>/camera_info</cameraInfoTopicName>
+        <imageTopicName>image</imageTopicName>
+        <cameraInfoTopicName>camera_info</cameraInfoTopicName>
         <frameName>camera_link</frameName>
         <hackBaseline>0.07</hackBaseline>

File: cssdbot_description/urdf/ur10e/ur10e.urdf.xacro (robot description, xacro)
@@ -405,10 +405,10 @@
       </camera>
       <plugin name="${prefix}camera_controller" filename="libgazebo_ros_camera.so">
-        <robotNamespace>$(arg robot_ns)</robotNamespace>
+        <robotNamespace></robotNamespace>
         <alwaysOn>true</alwaysOn>
         <updateRate>30</updateRate>
         <cameraName></cameraName>
-        <imageTopicName>/image</imageTopicName>
-        <cameraInfoTopicName>/camera_info</cameraInfoTopicName>
+        <imageTopicName>image</imageTopicName>
+        <cameraInfoTopicName>camera_info</cameraInfoTopicName>
         <frameName>camera_link</frameName>
         <hackBaseline>0.07</hackBaseline>

File: cssdbot_description/urdf/ur10e/ur10e_joint_limited_robot.urdf.xacro (robot description, xacro)
@@ -3,5 +3,4 @@
        name="ur10e" >
   <xacro:arg name="transmission_hw_interface" default="hardware_interface/PositionJointInterface"/>
-  <xacro:arg name="robot_ns" default=""/>
   <!-- common stuff -->
   <xacro:include filename="$(find cssdbot_description)/urdf/ur10e/common.gazebo.xacro" />
@@ -21,5 +20,5 @@
   <joint name="world_joint" type="fixed">
     <parent link="world" />
-    <child link = "${robot_ns}base_link" />
+    <child link = "base_link" />
     <origin xyz="0.0 0.0 0.0" rpy="0.0 0.0 0.0" />
   </joint>

File: cssdbot_description/urdf/ur10e/ur10e_robot.urdf.xacro (robot description, xacro)
@@ -5,8 +5,8 @@
   <!-- common stuff -->
   <xacro:include filename="$(find cssdbot_description)/urdf/ur10e/common.gazebo.xacro" />
-  <!-- ur10 -->
-  <xacro:include filename="$(find cssdbot_description)/urdf/ur10/ur10e.urdf.xacro" />
+  <!-- ur10e -->
+  <xacro:include filename="$(find cssdbot_description)/urdf/ur10e/ur10e.urdf.xacro" />
   <!-- arm -->
-  <xacro:ur10_robot prefix="" joint_limited="false"
+  <xacro:ur10e_robot prefix="" joint_limited="false"
     transmission_hw_interface="$(arg transmission_hw_interface)"
   />
