Commit message: added pointcloud perception. Not tested

File: cssdbot_description/urdf/ur10/ur10.urdf.xacro (robot description, xacro)
@@ -3,4 +3,5 @@
   <xacro:include filename="$(find cssdbot_description)/urdf/ur10/ur.transmission.xacro" />
   <xacro:include filename="$(find cssdbot_description)/urdf/ur10/ur.gazebo.xacro" />
+  <xacro:include filename="$(find realsense_gazebo_plugin)/urdf/realsense-D435.macro.xacro"/>
   <xacro:macro name="cylinder_inertial" params="radius length mass *origin">
     <inertial>
@@ -333,7 +334,7 @@
 -->
 <!--end of end effector-->
-<!-- start of camera -->
-  <joint name="camera_optical_joint" type="fixed">
+<!-- normal start of camera -->
     <!-- satisfy both gazebo convention and aruco pkg convetion. looking from x axis and z axis respectively. -->
+<!--  <joint name="camera_optical_joint" type="fixed">
     <origin xyz=" 0.055 0.06 0.0825" rpy="0 0.0 0" />>
     <parent link="${prefix}end_effector_link"/>
@@ -350,5 +351,4 @@
           <width>3840</width>
           <height>1080</height>
-          <!--<format>R8G8B8</format> -->
           <format>R8G8B8</format>
         </image>
@@ -359,7 +359,4 @@
         <noise>
           <type>gaussian</type>
-          <!-- Noise is sampled independently per pixel on each frame.
-               That pixel's noise value is added to each of its color
-               channels, which at that point lie in the range [0,1]. -->
           <mean>0.0</mean>
           <stddev>0.007</stddev>
@@ -381,7 +378,12 @@
       </plugin>
     </sensor>
-  </gazebo>
+  </gazebo> -->
 <!--camera link-->
-<!--end of camera link-->
+<!--end of normal camera link-->
+<!-- start of stero cam intel realsense-->
+    <xacro:realsense-D435 prefix="" parent="${prefix}end_effector_link">
+        <origin xyz="0.055 0.06 0.0825" rpy="0 0 0" />
+    </xacro:realsense-D435>
+<!-- end of stereo cam-->
     <!-- ROS base_link to UR 'Base' Coordinates transform -->
     <link name="${prefix}base"/>

Commit message: reverted realsense due to issue with two arms environment

File: cssdbot_description/urdf/ur10/ur10.urdf.xacro (robot description, xacro)
@@ -336,5 +336,5 @@
 <!-- normal start of camera -->
     <!-- satisfy both gazebo convention and aruco pkg convetion. looking from x axis and z axis respectively. -->
-<!--  <joint name="camera_optical_joint" type="fixed">
+ <joint name="camera_optical_joint" type="fixed">
     <origin xyz=" 0.055 0.06 0.0825" rpy="0 0.0 0" />>
     <parent link="${prefix}end_effector_link"/>
@@ -378,11 +378,12 @@
       </plugin>
     </sensor>
-  </gazebo> -->
+  </gazebo>
 <!--camera link-->
 <!--end of normal camera link-->
 <!-- start of stero cam intel realsense-->
+<!--
     <xacro:realsense-D435 prefix="" parent="${prefix}end_effector_link">
         <origin xyz="0.055 0.06 0.0825" rpy="0 0 0" />
-    </xacro:realsense-D435>
+    </xacro:realsense-D435> -->
 <!-- end of stereo cam-->
     <!-- ROS base_link to UR 'Base' Coordinates transform -->

Commit message: solved realsense camera namespace problems for both arms. Yet to remap topic names for arm.

File: cssdbot_description/urdf/ur10/ur10.urdf.xacro (robot description, xacro)
@@ -4,4 +4,5 @@
   <xacro:include filename="$(find cssdbot_description)/urdf/ur10/ur.gazebo.xacro" />
   <xacro:include filename="$(find realsense_gazebo_plugin)/urdf/realsense-D435.macro.xacro"/>
+  <xacro:arg name="camera_ns" default="arm" />
   <xacro:macro name="cylinder_inertial" params="radius length mass *origin">
     <inertial>
@@ -336,5 +337,5 @@
 <!-- normal start of camera -->
     <!-- satisfy both gazebo convention and aruco pkg convetion. looking from x axis and z axis respectively. -->
-<!--  <joint name="camera_optical_joint" type="fixed">
+ <!--<joint name="camera_optical_joint" type="fixed">
     <origin xyz=" 0.055 0.06 0.0825" rpy="0 0.0 0" />>
     <parent link="${prefix}end_effector_link"/>
@@ -382,6 +383,6 @@
 <!--end of normal camera link-->
 <!-- start of stero cam intel realsense-->
-    <xacro:realsense-D435 prefix="" parent="${prefix}end_effector_link">
-        <origin xyz="0.055 0.06 0.0825" rpy="0 0 0" />
+    <xacro:realsense-D435 prefix="$(arg camera_ns)" parent="${prefix}end_effector_link">
+        <origin xyz="0.045 0.06 0.09" rpy="0 0 0" />
     </xacro:realsense-D435>
 <!-- end of stereo cam-->

File: cssdbot_description/urdf/ur10e/ur10e.urdf.xacro (robot description, xacro)
@@ -3,4 +3,5 @@
   <xacro:include filename="$(find cssdbot_description)/urdf/ur10e/ur.transmission.xacro" />
   <xacro:include filename="$(find cssdbot_description)/urdf/ur10e/ur.gazebo.xacro" />
+  <xacro:include filename="$(find realsense_gazebo_plugin)/urdf/realsense-D435.macro.xacro"/>
   <xacro:macro name="cylinder_inertial" params="radius length mass *origin">
     <inertial>
@@ -372,6 +373,7 @@
 <!--end of end effector-->
 <!-- start of camera -->
+    <!-- satisfy both gazebo convention and aruco pkg convetion. looking from x axis and z axis respectively. -->
+<!--
   <joint name="${prefix}camera_optical_joint" type="fixed">
-    <!-- satisfy both gazebo convention and aruco pkg convetion. looking from x axis and z axis respectively. -->
     <origin xyz=" 0.055 0.06 0.0825" rpy="0 0.0 0" />>
     <parent link="${prefix}end_effector_link"/>
@@ -388,5 +390,4 @@
           <width>3840</width>
           <height>1080</height>
-          <!--<format>R8G8B8</format> -->
           <format>R8G8B8</format>
         </image>
@@ -397,7 +398,4 @@
         <noise>
           <type>gaussian</type>
-          <!-- Noise is sampled independently per pixel on each frame.
-               That pixel's noise value is added to each of its color
-               channels, which at that point lie in the range [0,1]. -->
           <mean>0.0</mean>
           <stddev>0.007</stddev>
@@ -420,7 +418,12 @@
       </plugin>
     </sensor>
-  </gazebo>
+  </gazebo> -->
 <!--camera link-->
 <!--end of camera link-->
+<!-- start of stero cam intel realsense-->
+    <xacro:realsense-D435 prefix="$(arg camera_ns)" parent="${prefix}end_effector_link">
+        <origin xyz="0.055 0.06 0.0825" rpy="0 0 0" />
+    </xacro:realsense-D435>
+<!-- end of stereo cam-->
     <!-- ROS base_link to UR 'Base' Coordinates transform -->
     <link name="${prefix}base"/>

Commit message: unable to have namespace for gazebo realsense plugin. Revert gazebo back to normal camera, and allowed demo.launch to accommodate 2 different types of camera situation

File: cssdbot_description/urdf/ur10/ur10.urdf.xacro (robot description, xacro)
@@ -337,5 +337,5 @@
 <!-- normal start of camera -->
     <!-- satisfy both gazebo convention and aruco pkg convetion. looking from x axis and z axis respectively. -->
- <!--<joint name="camera_optical_joint" type="fixed">
+ <joint name="camera_optical_joint" type="fixed">
     <origin xyz=" 0.055 0.06 0.0825" rpy="0 0.0 0" />>
     <parent link="${prefix}end_effector_link"/>
@@ -379,12 +379,7 @@
       </plugin>
     </sensor>
-  </gazebo> -->
+  </gazebo>
 <!--camera link-->
 <!--end of normal camera link-->
-<!-- start of stero cam intel realsense-->
-    <xacro:realsense-D435 prefix="$(arg camera_ns)" parent="${prefix}end_effector_link">
-        <origin xyz="0.045 0.06 0.09" rpy="0 0 0" />
-    </xacro:realsense-D435>
-<!-- end of stereo cam-->
     <!-- ROS base_link to UR 'Base' Coordinates transform -->
     <link name="${prefix}base"/>

File: cssdbot_description/urdf/ur10e/ur10e.urdf.xacro (robot description, xacro)
@@ -374,5 +374,4 @@
 <!-- start of camera -->
     <!-- satisfy both gazebo convention and aruco pkg convetion. looking from x axis and z axis respectively. -->
-<!--
   <joint name="${prefix}camera_optical_joint" type="fixed">
     <origin xyz=" 0.055 0.06 0.0825" rpy="0 0.0 0" />>
@@ -418,12 +417,7 @@
       </plugin>
     </sensor>
-  </gazebo> -->
+  </gazebo>
 <!--camera link-->
 <!--end of camera link-->
-<!-- start of stero cam intel realsense-->
-    <xacro:realsense-D435 prefix="$(arg camera_ns)" parent="${prefix}end_effector_link">
-        <origin xyz="0.055 0.06 0.0825" rpy="0 0 0" />
-    </xacro:realsense-D435>
-<!-- end of stereo cam-->
     <!-- ROS base_link to UR 'Base' Coordinates transform -->
     <link name="${prefix}base"/>
