Commit message: cleanup codes, fix issue on cam scanning, tested on gazebo!

File: cssdbot_description/urdf/ur10/ur10.urdf.xacro (robot description, xacro)
@@ -1,7 +1,7 @@
-<?xml version="1.0" ?>
+<?xml version="1.0"?>
 <robot xmlns:xacro="http://wiki.ros.org/xacro">
   <xacro:include filename="$(find cssdbot_description)/urdf/ur10/ur.transmission.xacro" />
   <xacro:include filename="$(find cssdbot_description)/urdf/ur10/ur.gazebo.xacro" />
-  <xacro:include filename="$(find realsense_gazebo_plugin)/urdf/realsense-D435.macro.xacro" />
+  <!-- <xacro:include filename="$(find realsense_gazebo_plugin)/urdf/realsense-D435.macro.xacro"/> -->
   <xacro:arg name="camera_ns" default="arm" />
   <xacro:macro name="cylinder_inertial" params="radius length mass *origin">
@@ -9,5 +9,7 @@
       <mass value="${mass}" />
       <xacro:insert_block name="origin" />
-      <inertia ixx="${0.0833333 * mass * (3 * radius * radius + length * length)}" ixy="0.0" ixz="0.0" iyy="${0.0833333 * mass * (3 * radius * radius + length * length)}" iyz="0.0" izz="${0.5 * mass * radius * radius}" />
+      <inertia ixx="${0.0833333 * mass * (3 * radius * radius + length * length)}" ixy="0.0" ixz="0.0"
+        iyy="${0.0833333 * mass * (3 * radius * radius + length * length)}" iyz="0.0"
+        izz="${0.5 * mass * radius * radius}" />
     </inertial>
   </xacro:macro>
@@ -21,5 +23,5 @@
     transmission_hw_interface:=hardware_interface/PositionJointInterface">
     <!-- Inertia parameters -->
-    <xacro:property name="base_mass" value="4.0" /> <!-- This mass might be incorrect -->
+    <xacro:property name="base_mass" value="4.0" />  <!-- This mass might be incorrect -->
     <xacro:property name="shoulder_mass" value="7.778" />
     <xacro:property name="upper_arm_mass" value="12.93" />
@@ -47,5 +49,5 @@
     <xacro:property name="d6" value="0.0922" />
     <!-- Arbitrary offsets for shoulder/elbow joints -->
-    <xacro:property name="shoulder_offset" value="0.220941" /> <!-- measured from model -->
+    <xacro:property name="shoulder_offset" value="0.220941" />  <!-- measured from model -->
     <xacro:property name="elbow_offset" value="-0.1719" /> <!-- measured from model -->
     <!-- link lengths used in model -->
@@ -56,16 +58,16 @@
     <xacro:property name="wrist_2_length" value="${d5}" />
     <xacro:property name="wrist_3_length" value="${d6}" />
-    <link name="${prefix}base_link">
-      <visual>
-        <geometry>
-          <mesh filename="package://cssdbot_description/meshes/ur10/visual/base.dae" />
-        </geometry>
-        <material name="LightGrey">
-          <color rgba="0.7 0.7 0.7 1.0" />
-        </material>
-      </visual>
-      <collision>
-        <geometry>
-          <mesh filename="package://cssdbot_description/meshes/ur10/collision/base.stl" />
+    <link name="${prefix}base_link" >
+      <visual>
+        <geometry>
+          <mesh filename="package://cssdbot_description/meshes/ur10/visual/base.dae"/>
+        </geometry>
+        <material name="LightGrey">
+          <color rgba="0.7 0.7 0.7 1.0"/>
+        </material>
+      </visual>
+      <collision>
+        <geometry>
+          <mesh filename="package://cssdbot_description/meshes/ur10/collision/base.stl"/>
         </geometry>
       </collision>
@@ -76,27 +78,27 @@
     <joint name="${prefix}shoulder_pan_joint" type="revolute">
       <parent link="${prefix}base_link" />
-      <child link="${prefix}shoulder_link" />
+      <child link = "${prefix}shoulder_link" />
       <origin xyz="0.0 0.0 ${shoulder_height}" rpy="0.0 0.0 0.0" />
       <axis xyz="0 0 1" />
       <xacro:unless value="${joint_limited}">
-        <limit lower="${-2.0 * pi}" upper="${2.0 * pi}" effort="330.0" velocity="2.16" />
-      </xacro:unless>
-      <xacro:if value="${joint_limited}">
-        <limit lower="${shoulder_pan_lower_limit}" upper="${shoulder_pan_upper_limit}" effort="330.0" velocity="2.16" />
-      </xacro:if>
-      <dynamics damping="0.0" friction="0.0" />
+        <limit lower="${-2.0 * pi}" upper="${2.0 * pi}" effort="330.0" velocity="2.16"/>
+      </xacro:unless>
+      <xacro:if value="${joint_limited}">
+        <limit lower="${shoulder_pan_lower_limit}" upper="${shoulder_pan_upper_limit}" effort="330.0" velocity="2.16"/>
+      </xacro:if>
+      <dynamics damping="0.0" friction="0.0"/>
     </joint>
     <link name="${prefix}shoulder_link">
       <visual>
         <geometry>
-          <mesh filename="package://cssdbot_description/meshes/ur10/visual/shoulder.dae" />
-        </geometry>
-        <material name="LightGrey">
-          <color rgba="0.7 0.7 0.7 1.0" />
-        </material>
-      </visual>
-      <collision>
-        <geometry>
-          <mesh filename="package://cssdbot_description/meshes/ur10/collision/shoulder.stl" />
+          <mesh filename="package://cssdbot_description/meshes/ur10/visual/shoulder.dae"/>
+        </geometry>
+        <material name="LightGrey">
+          <color rgba="0.7 0.7 0.7 1.0"/>
+        </material>
+      </visual>
+      <collision>
+        <geometry>
+          <mesh filename="package://cssdbot_description/meshes/ur10/collision/shoulder.stl"/>
         </geometry>
       </collision>
@@ -107,27 +109,27 @@
     <joint name="${prefix}shoulder_lift_joint" type="revolute">
       <parent link="${prefix}shoulder_link" />
-      <child link="${prefix}upper_arm_link" />
+      <child link = "${prefix}upper_arm_link" />
       <origin xyz="0.0 ${shoulder_offset} 0.0" rpy="0.0 ${pi / 2.0} 0.0" />
       <axis xyz="0 1 0" />
       <xacro:unless value="${joint_limited}">
-        <limit lower="${-2.0 * pi}" upper="${2.0 * pi}" effort="330.0" velocity="2.16" />
-      </xacro:unless>
-      <xacro:if value="${joint_limited}">
-        <limit lower="${shoulder_lift_lower_limit}" upper="${shoulder_lift_upper_limit}" effort="330.0" velocity="2.16" />
-      </xacro:if>
-      <dynamics damping="0.0" friction="0.0" />
+        <limit lower="${-2.0 * pi}" upper="${2.0 * pi}" effort="330.0" velocity="2.16"/>
+      </xacro:unless>
+      <xacro:if value="${joint_limited}">
+        <limit lower="${shoulder_lift_lower_limit}" upper="${shoulder_lift_upper_limit}" effort="330.0" velocity="2.16"/>
+      </xacro:if>
+      <dynamics damping="0.0" friction="0.0"/>
     </joint>
     <link name="${prefix}upper_arm_link">
       <visual>
         <geometry>
-          <mesh filename="package://cssdbot_description/meshes/ur10/visual/upperarm.dae" />
-        </geometry>
-        <material name="LightGrey">
-          <color rgba="0.7 0.7 0.7 1.0" />
-        </material>
-      </visual>
-      <collision>
-        <geometry>
-          <mesh filename="package://cssdbot_description/meshes/ur10/collision/upperarm.stl" />
+          <mesh filename="package://cssdbot_description/meshes/ur10/visual/upperarm.dae"/>
+        </geometry>
+        <material name="LightGrey">
+          <color rgba="0.7 0.7 0.7 1.0"/>
+        </material>
+      </visual>
+      <collision>
+        <geometry>
+          <mesh filename="package://cssdbot_description/meshes/ur10/collision/upperarm.stl"/>
         </geometry>
       </collision>
@@ -138,27 +140,27 @@
     <joint name="${prefix}elbow_joint" type="revolute">
       <parent link="${prefix}upper_arm_link" />
-      <child link="${prefix}forearm_link" />
+      <child link = "${prefix}forearm_link" />
       <origin xyz="0.0 ${elbow_offset} ${upper_arm_length}" rpy="0.0 0.0 0.0" />
       <axis xyz="0 1 0" />
       <xacro:unless value="${joint_limited}">
-        <limit lower="${-pi}" upper="${pi}" effort="150.0" velocity="3.15" />
-      </xacro:unless>
-      <xacro:if value="${joint_limited}">
-        <limit lower="${elbow_joint_lower_limit}" upper="${elbow_joint_upper_limit}" effort="150.0" velocity="3.15" />
-      </xacro:if>
-      <dynamics damping="0.0" friction="0.0" />
+        <limit lower="${-pi}" upper="${pi}" effort="150.0" velocity="3.15"/>
+      </xacro:unless>
+      <xacro:if value="${joint_limited}">
+        <limit lower="${elbow_joint_lower_limit}" upper="${elbow_joint_upper_limit}" effort="150.0" velocity="3.15"/>
+      </xacro:if>
+      <dynamics damping="0.0" friction="0.0"/>
     </joint>
     <link name="${prefix}forearm_link">
       <visual>
-        <geometry>
-          <mesh filename="package://cssdbot_description/meshes/ur10/visual/forearm.dae" />
-        </geometry>
-        <material name="LightGrey">
-          <color rgba="0.7 0.7 0.7 1.0" />
-        </material>
-      </visual>
-      <collision>
-        <geometry>
-          <mesh filename="package://cssdbot_description/meshes/ur10/collision/forearm.stl" />
+         <geometry>
+          <mesh filename="package://cssdbot_description/meshes/ur10/visual/forearm.dae"/>
+        </geometry>
+        <material name="LightGrey">
+          <color rgba="0.7 0.7 0.7 1.0"/>
+        </material>
+      </visual>
+      <collision>
+        <geometry>
+          <mesh filename="package://cssdbot_description/meshes/ur10/collision/forearm.stl"/>
         </geometry>
       </collision>
@@ -169,27 +171,27 @@
     <joint name="${prefix}wrist_1_joint" type="revolute">
       <parent link="${prefix}forearm_link" />
-      <child link="${prefix}wrist_1_link" />
+      <child link = "${prefix}wrist_1_link" />
       <origin xyz="0.0 0.0 ${forearm_length}" rpy="0.0 ${pi / 2.0} 0.0" />
       <axis xyz="0 1 0" />
       <xacro:unless value="${joint_limited}">
-        <limit lower="${-2.0 * pi}" upper="${2.0 * pi}" effort="54.0" velocity="3.2" />
-      </xacro:unless>
-      <xacro:if value="${joint_limited}">
-        <limit lower="${wrist_1_lower_limit}" upper="${wrist_1_upper_limit}" effort="54.0" velocity="3.2" />
-      </xacro:if>
-      <dynamics damping="0.0" friction="0.0" />
+        <limit lower="${-2.0 * pi}" upper="${2.0 * pi}" effort="54.0" velocity="3.2"/>
+      </xacro:unless>
+      <xacro:if value="${joint_limited}">
+        <limit lower="${wrist_1_lower_limit}" upper="${wrist_1_upper_limit}" effort="54.0" velocity="3.2"/>
+      </xacro:if>
+      <dynamics damping="0.0" friction="0.0"/>
     </joint>
     <link name="${prefix}wrist_1_link">
       <visual>
         <geometry>
-          <mesh filename="package://cssdbot_description/meshes/ur10/visual/wrist1.dae" />
-        </geometry>
-        <material name="LightGrey">
-          <color rgba="0.7 0.7 0.7 1.0" />
-        </material>
-      </visual>
-      <collision>
-        <geometry>
-          <mesh filename="package://cssdbot_description/meshes/ur10/collision/wrist1.stl" />
+          <mesh filename="package://cssdbot_description/meshes/ur10/visual/wrist1.dae"/>
+        </geometry>
+        <material name="LightGrey">
+          <color rgba="0.7 0.7 0.7 1.0"/>
+        </material>
+      </visual>
+      <collision>
+        <geometry>
+          <mesh filename="package://cssdbot_description/meshes/ur10/collision/wrist1.stl"/>
         </geometry>
       </collision>
@@ -200,27 +202,27 @@
     <joint name="${prefix}wrist_2_joint" type="revolute">
       <parent link="${prefix}wrist_1_link" />
-      <child link="${prefix}wrist_2_link" />
+      <child link = "${prefix}wrist_2_link" />
       <origin xyz="0.0 ${wrist_1_length} 0.0" rpy="0.0 0.0 0.0" />
       <axis xyz="0 0 1" />
       <xacro:unless value="${joint_limited}">
-        <limit lower="${-2.0 * pi}" upper="${2.0 * pi}" effort="54.0" velocity="3.2" />
-      </xacro:unless>
-      <xacro:if value="${joint_limited}">
-        <limit lower="${wrist_2_lower_limit}" upper="${wrist_2_upper_limit}" effort="54.0" velocity="3.2" />
-      </xacro:if>
-      <dynamics damping="0.0" friction="0.0" />
+        <limit lower="${-2.0 * pi}" upper="${2.0 * pi}" effort="54.0" velocity="3.2"/>
+      </xacro:unless>
+      <xacro:if value="${joint_limited}">
+        <limit lower="${wrist_2_lower_limit}" upper="${wrist_2_upper_limit}" effort="54.0" velocity="3.2"/>
+      </xacro:if>
+      <dynamics damping="0.0" friction="0.0"/>
     </joint>
     <link name="${prefix}wrist_2_link">
       <visual>
         <geometry>
-          <mesh filename="package://cssdbot_description/meshes/ur10/visual/wrist2.dae" />
-        </geometry>
-        <material name="LightGrey">
-          <color rgba="0.7 0.7 0.7 1.0" />
-        </material>
-      </visual>
-      <collision>
-        <geometry>
-          <mesh filename="package://cssdbot_description/meshes/ur10/collision/wrist2.stl" />
+          <mesh filename="package://cssdbot_description/meshes/ur10/visual/wrist2.dae"/>
+        </geometry>
+        <material name="LightGrey">
+          <color rgba="0.7 0.7 0.7 1.0"/>
+        </material>
+      </visual>
+      <collision>
+        <geometry>
+          <mesh filename="package://cssdbot_description/meshes/ur10/collision/wrist2.stl"/>
         </geometry>
       </collision>
@@ -231,27 +233,27 @@
     <joint name="${prefix}wrist_3_joint" type="revolute">
       <parent link="${prefix}wrist_2_link" />
-      <child link="${prefix}wrist_3_link" />
+      <child link = "${prefix}wrist_3_link" />
       <origin xyz="0.0 0.0 ${wrist_2_length}" rpy="0.0 0.0 0.0" />
       <axis xyz="0 1 0" />
       <xacro:unless value="${joint_limited}">
-        <limit lower="${-2.0 * pi}" upper="${2.0 * pi}" effort="54.0" velocity="3.2" />
-      </xacro:unless>
-      <xacro:if value="${joint_limited}">
-        <limit lower="${wrist_3_lower_limit}" upper="${wrist_3_upper_limit}" effort="54.0" velocity="3.2" />
-      </xacro:if>
-      <dynamics damping="0.0" friction="0.0" />
+        <limit lower="${-2.0 * pi}" upper="${2.0 * pi}" effort="54.0" velocity="3.2"/>
+      </xacro:unless>
+      <xacro:if value="${joint_limited}">
+        <limit lower="${wrist_3_lower_limit}" upper="${wrist_3_upper_limit}" effort="54.0" velocity="3.2"/>
+      </xacro:if>
+      <dynamics damping="0.0" friction="0.0"/>
     </joint>
     <link name="${prefix}wrist_3_link">
       <visual>
         <geometry>
-          <mesh filename="package://cssdbot_description/meshes/ur10/visual/wrist3.dae" />
-        </geometry>
-        <material name="LightGrey">
-          <color rgba="0.7 0.7 0.7 1.0" />
-        </material>
-      </visual>
-      <collision>
-        <geometry>
-          <mesh filename="package://cssdbot_description/meshes/ur10/collision/wrist3.stl" />
+          <mesh filename="package://cssdbot_description/meshes/ur10/visual/wrist3.dae"/>
+        </geometry>
+        <material name="LightGrey">
+          <color rgba="0.7 0.7 0.7 1.0"/>
+        </material>
+      </visual>
+      <collision>
+        <geometry>
+          <mesh filename="package://cssdbot_description/meshes/ur10/collision/wrist3.stl"/>
         </geometry>
       </collision>
@@ -262,5 +264,5 @@
     <joint name="${prefix}ee_fixed_joint" type="fixed">
       <parent link="${prefix}wrist_3_link" />
-      <child link="${prefix}ee_link" />
+      <child link = "${prefix}ee_link" />
       <origin xyz="0.0 ${wrist_3_length} 0.0" rpy="0.0 0.0 ${pi/2.0}" />
     </joint>
@@ -268,13 +270,13 @@
       <collision>
         <geometry>
-          <box size="0.01 0.01 0.01" />
-        </geometry>
-        <origin rpy="0 0 0" xyz="-0.01 0 0" />
-      </collision>
-    </link>
-    <!--end effector-->
-    <joint name="${prefix}end_effector_joint" type="fixed">
+          <box size="0.01 0.01 0.01"/>
+        </geometry>
+        <origin rpy="0 0 0" xyz="-0.01 0 0"/>
+      </collision>
+    </link>
+  <!--end effector-->
+  <joint name="${prefix}end_effector_joint" type="fixed">
       <parent link="${prefix}ee_link" />
-      <child link="${prefix}end_effector_link" />
+      <child link = "${prefix}end_effector_link" />
       <origin xyz="0.0 0.0 0.0" rpy="0.0 0 0.0" />
     </joint>
@@ -282,23 +284,35 @@
       <visual>
         <geometry>
-          <mesh filename="package://cssdbot_description/meshes/end_effector/visual/end_effector.STL" scale="0.001 0.001 0.001" />
+          <mesh filename="package://cssdbot_description/meshes/end_effector/visual/end_effector.STL" scale = "0.001 0.001 0.001"/>
         </geometry>
         <origin xyz="0.0 0.0 0.0" rpy="3.14 0 0" />
         <material name="LightGrey">
-          <color rgba="0.7 0.7 0.7 1.0" />
-        </material>
-      </visual>
-      <collision>
-        <geometry>
-          <mesh filename="package://cssdbot_description/meshes/end_effector/collision/end_effector_holes.stl" scale="1 1 1" />
+          <color rgba="0.7 0.7 0.7 1.0"/>
+        </material>
+      </visual>
+      <collision>
+        <geometry>
+          <mesh filename="package://cssdbot_description/meshes/end_effector/collision/end_effector_holes.stl" scale = "1 1 1"/>
         </geometry>
         <origin xyz="0.0 0.0 0.0" rpy="3.14 0 0" />
+        <surface>
+          <contact>
+            <ode>
+              <kp>1000000.0</kp>
+              <kd>1.0</kd>
+              <mu1>0.8</mu1>
+              <mu2>0.8</mu2>
+              <maxVel>0.0</maxVel>
+              <minDepth>0.001</minDepth>
+            </ode>
+          </contact>
+        </surface>
       </collision>
       <!-- Extents: ([0.0125, 0.2112], +/- 0.05673, [-0.046, -0.043]) -->
       <!-- Note: I'm making this 3mm thicker than the actual model -->
       <collision>
-        <origin xyz="0.11185 0.0 0.046" />
-        <geometry>
-          <box size="0.1987 0.11346 0.006" />
+        <origin xyz="0.11185 0.0 0.046"/>
+        <geometry>
+          <box size="0.1987 0.11346 0.006"/>
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
File: cssdbot_description/urdf/ur10e/ur10e.urdf.xacro (robot description, xacro)
@@ -3,5 +3,5 @@
   <xacro:include filename="$(find cssdbot_description)/urdf/ur10e/ur.transmission.xacro" />
   <xacro:include filename="$(find cssdbot_description)/urdf/ur10e/ur.gazebo.xacro" />
-  <xacro:include filename="$(find realsense_gazebo_plugin)/urdf/realsense-D435.macro.xacro"/>
+  <!-- <xacro:include filename="$(find realsense_gazebo_plugin)/urdf/realsense-D435.macro.xacro"/> -->
   <xacro:macro name="cylinder_inertial" params="radius length mass *origin">
     <inertial>
@@ -332,5 +332,17 @@
           <mesh filename="package://cssdbot_description/meshes/end_effector/collision/end_effector_holes.stl" scale = "1 1 1"/>
         </geometry>
-	      <origin xyz="0.0 0.0 0.0" rpy="3.14 0 0" />
+        <origin xyz="0.0 0.0 0.0" rpy="3.14 0 0" />
+        <surface>
+          <contact>
+            <ode>
+              <kp>1000000.0</kp>
+              <kd>1.0</kd>
+              <mu1>0.8</mu1>
+              <mu2>0.8</mu2>
+              <maxVel>0.0</maxVel>
+              <minDepth>0.001</minDepth>
+            </ode>
+          </contact>
+        </surface>
       </collision>
       <!-- Extents: ([0.0125, 0.2112], +/- 0.05673, [-0.046, -0.043]) -->
