Commit message: FIXED GAZEBO CONTROLLER LAUNCHgit add -Agit add -A!(launch files are very unhealthy)

File: cssdbot_description/urdf/ur10e/ur10e_robot.urdf.xacro (robot description, xacro)
@@ -2,4 +2,5 @@
 <robot xmlns:xacro="http://ros.org/wiki/xacro"
        name="ur10e" >
+  <xacro:arg name="transmission_hw_interface" default="hardware_interface/PositionJointInterface"/>
   <!-- common stuff -->
   <xacro:include filename="$(find cssdbot_description)/urdf/ur10e/common.gazebo.xacro" />
@@ -7,10 +8,12 @@
   <xacro:include filename="$(find cssdbot_description)/urdf/ur10e/ur10e.urdf.xacro" />
   <!-- arm -->
-  <xacro:ur10e_robot prefix="" joint_limited="false" />
+  <xacro:ur10e_robot prefix="" joint_limited="false"
+  transmission_hw_interface="$(arg transmission_hw_interface)"
+  />
   <link name="world" />
   <joint name="world_joint" type="fixed">
     <parent link="world" />
     <child link = "base_link" />
-    <origin xyz="0.0 0.0 0.0" rpy="0.0 0.0 0.0" />
+    <origin xyz="0.0 0.0 0.005" rpy="0.0 0.0 0.0" />
   </joint>
 </robot>
